File: ds_test_board/ds_test.kicad_pcb (KiCad board)
At the start: 2 copper layers, 63 parts, among them J2 DF40C-60DP-0.4V_51_, J3 Conn_01x30, J4 Conn_01x30

Commit message: 1201
Parts:
- added REF**: MountingHole_2.5mm_Pad_TopBottom, MountingHole:MountingHole_2.5mm_Pad_TopBottom, F.Cu at (125.7, 61.0)
- added REF**: MountingHole_2.5mm_Pad_TopBottom, MountingHole:MountingHole_2.5mm_Pad_TopBottom, F.Cu at (125.7, 118.1)
- added REF**: MountingHole_2.5mm_Pad_TopBottom, MountingHole:MountingHole_2.5mm_Pad_TopBottom, F.Cu at (209.6, 61.0)
- added REF**: MountingHole_2.5mm_Pad_TopBottom, MountingHole:MountingHole_2.5mm_Pad_TopBottom, F.Cu at (209.6, 118.4)
- added TP61: TestPoint, TestPoint:TestPoint_THTPad_1.5x1.5mm_Drill0.7mm, F.Cu at (125.5, 67.3)
- added TP62: TestPoint, TestPoint:TestPoint_THTPad_1.5x1.5mm_Drill0.7mm, F.Cu at (125.7, 112.0)
- added TP63: TestPoint, TestPoint:TestPoint_THTPad_1.5x1.5mm_Drill0.7mm, F.Cu at (209.7, 67.3)
- added TP64: TestPoint, TestPoint:TestPoint_THTPad_1.5x1.5mm_Drill0.7mm, F.Cu at (209.6, 112.0)
- J2: moved to B.Cu
- TP1, TP10, TP11, TP12, TP13, TP14, TP15, TP16, TP17, TP18, TP19, TP2, TP20, TP21, TP22, TP23, TP24, TP25, TP26, TP27, TP28, TP29, TP3, TP30, TP31, TP32, TP33, TP34, TP35, TP36, TP37, TP38, TP39, TP4, TP40, TP41, TP42, TP43, TP44, TP45, TP46, TP47, TP48, TP49, TP5, TP50, TP51, TP52, TP53, TP54, TP55, TP56, TP57, TP58, TP59, TP6, TP60, TP7, TP8, TP9: footprint TestPoint:TestPoint_Pad_1.5x1.5mm -> TestPoint:TestPoint_THTPad_1.5x1.5mm_Drill0.7mm
- moved TP27 99.4 mm to (138.4, 61.2)
- moved TP26 91.8 mm to (140.9, 67.3)
- moved TP25 91.1 mm to (143.5, 61.2)
- moved TP24 83.7 mm to (146.0, 67.3)
- moved TP23 82.9 mm to (148.6, 61.2)
- moved TP22 75.8 mm to (151.1, 67.3)
- moved TP17 75.5 mm to (163.8, 61.2)
- moved TP18 75.4 mm to (161.3, 67.3)
- moved TP21 74.9 mm to (153.6, 61.2)
- moved TP20 68.1 mm to (156.2, 67.3)
- moved TP38 67.4 mm to (186.7, 118.6)
- moved TP19 67.0 mm to (158.7, 61.2)
- moved TP15 66.9 mm to (168.9, 61.2)
- moved TP16 66.8 mm to (166.3, 67.3)
- moved TP9 65.4 mm to (184.1, 61.2)
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Connections:
- net GND renamed /GND
Routing:
- net /GND: track 0.00 -> 616.6 mm
- net +5V: track 0.00 -> 297.3 mm
- net /VCCIO2/3: track 0.00 -> 126.4 mm
- net +3V3: track 0.00 -> 105.1 mm
- net +2V5: track 0.00 -> 96.1 mm
- net /VDD_1V8: track 0.00 -> 83.7 mm
- net /IOB4A: track 0.00 -> 66.5 mm
- net /IOR18A: track 0.00 -> 65.3 mm
- net /M0_D0P: track 0.00 -> 64.4 mm
- net /IOB26A: track 0.00 -> 61.9 mm
- net /IOR20A: track 0.00 -> 60.9 mm
- net /M0_D1N: track 0.00 -> 59.9 mm
- net /IOB24A: track 0.00 -> 57.4 mm
- net /M0_D0N: track 0.00 -> 57.4 mm
- net /IOR22A: track 0.00 -> 56.6 mm
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Other:
- board outline added: 91.4 x 64.8 mm
