File: base_board1/base_board1.kicad_pcb (KiCad board)
At the start: 2 copper layers, 91.4 x 100 mm, 203 parts, among them J1 DF40C-60DP-0.4V_51_, J2 DF40C-60DP-0.4V_51_, J3 Conn_01x30, J4 Conn_01x30, J5 Conn_01x30, J6 Conn_01x30

Commit message: 1218
Parts:
- removed the REF** at (128.5, 146.3)
- removed the REF** at (125.7, 79.2)
- removed the REF** at (210.2, 134.6)
- removed the REF** at (125.7, 136.6)
- removed the REF** at (129.0, 120.4)
- removed the REF** at (125.7, 130.6)
- removed the REF** at (208.1, 119.0)
- removed the REF** at (126.5, 66.7)
- removed the REF** at (209.7, 82.9)
- removed the REF** at (169.5, 59.4)
- removed the REF** at (159.3, 59.4)
- removed the REF** at (160.6, 154.7)
- removed the REF** at (139.7, 154.7)
- removed the REF** at (197.9, 154.7)
- removed the REF** at (137.2, 59.4)
- removed the REF** at (192.7, 59.4)
- removed the REF** at (185.2, 59.4)
- removed the REF** at (180.3, 154.7)
- removed the REF** at (178.0, 59.4)
- removed the REF** at (205.1, 67.4)
- removed the REF** at (201.0, 59.4)
- removed TP10, TP111, TP128, TP13, TP16, TP21, TP4, TP61, TP63, TP66, TP7, TP81, TP93: TestPoint, TestPoint:TestPoint_THTPad_1.5x1.5mm_Drill0.7mm
- removed TP116, TP127, TP62, TP64, TP65, TP68, TP94: TestPoint, TestPoint:TestPoint_Pad_1.5x1.5mm
- TP101, TP103, TP105, TP107, TP109, TP113, TP115, TP117, TP119, TP121, TP123, TP69, TP71, TP73, TP75, TP77, TP79, TP83, TP85, TP87, TP89, TP91, TP95, TP99: footprint TestPoint:TestPoint_THTPad_1.5x1.5mm_Drill0.7mm -> TestPoint:TestPoint_Pad_1.5x1.5mm
- TP35, TP37: footprint TestPoint:TestPoint_THTPad_2.0x2.0mm_Drill1.0mm -> TestPoint:TestPoint_Pad_1.5x1.5mm
- moved REF** 8.00 mm to (217.6, 61.0)
- moved REF** 8.00 mm to (217.6, 152.9)
- moved REF** 4.00 mm to (128.5, 113.3)
- moved REF** 4.00 mm to (128.5, 110.7)
- moved REF** 4.00 mm to (128.5, 100.6)
- moved REF** 4.00 mm to (128.5, 115.8)
- moved REF** 4.00 mm to (128.5, 95.5)
- moved REF** 4.00 mm to (128.5, 105.7)
- moved REF** 4.00 mm to (128.5, 103.1)
- moved REF** 4.00 mm to (128.5, 118.4)
- moved REF** 4.00 mm to (128.5, 108.2)
- moved REF** 4.00 mm to (128.5, 98.0)
- moved J1 4.00 mm to (172.6, 113.0)
- moved J2 4.00 mm to (172.5, 99.0)
- moved J3 4.00 mm to (171.6, 80.5)
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Connections:
- J1 pad 61: Net-(J1-Pad61) -> unconnected-(J1-Pad61)
- J1 pad 62: Net-(J1-Pad62) -> unconnected-(J1-Pad62)
- J1 pad 63: Net-(J1-Pad63) -> unconnected-(J1-Pad63)
- J1 pad 64: Net-(J1-Pad64) -> unconnected-(J1-Pad64)
Routing:
- net GND: track 1267.3 -> 8.90 mm, vias 7 -> 0
- net Net-(J1-Pad63): track 58.0 -> 0.00 mm
- net Net-(J1-Pad61): track 56.0 -> 0.00 mm, vias 1 -> 0
- net Net-(J1-Pad62): track 54.7 -> 0.00 mm
- net Net-(J1-Pad64): track 52.7 -> 0.00 mm, vias 1 -> 0
Other:
- board size 91.4 x 100 mm -> 99.4 x 100 mm

Commit message: 1218
Parts:
- J1, J2: value DF40C-60DP-0.4V_51_ -> DF40C-60DS-0.4V_51_; footprint SamacSys_Parts:DF40C-60DP-0.4V_51_ -> samacsys:DF40C60DS04V51
- TP101, TP103, TP105, TP107, TP109, TP113, TP115, TP117, TP119, TP121, TP123, TP69, TP71, TP73, TP75, TP77, TP79, TP83, TP85, TP87, TP89, TP91, TP95, TP99: footprint TestPoint:TestPoint_Pad_1.5x1.5mm -> TestPoint:TestPoint_THTPad_1.5x1.5mm_Drill0.7mm
Connections:
- J1 pad 1: GND -> /GND
- J1 pad 15: GND -> /GND
- J1 pad 2: GND -> /GND
- J1 pad 27: GND -> /GND
- J1 pad 28: GND -> /GND
- J1 pad 45: GND -> /GND
- J1 pad 50: GND -> /GND
- J1 pad 59: GND -> /GND
- J1 pad 60: GND -> /GND
- J2 pad 1: GND -> /GND
- J2 pad 19: GND -> /GND
- J2 pad 29: GND -> /GND
- J2 pad 35: GND -> /GND
- J2 pad 41: GND -> /GND
- J2 pad 47: GND -> /GND
- J2 pad 53: GND -> /GND
- J2 pad 59: GND -> /GND
- J4 pad 1: GND -> /GND
- J4 pad 10: GND -> /GND
- J4 pad 13: GND -> /GND
- J4 pad 16: GND -> /GND
- J4 pad 21: GND -> /GND
- J4 pad 30: GND -> /GND
- J4 pad 4: GND -> /GND
- J4 pad 7: GND -> /GND
- J5 pad 1: GND -> /GND
- J5 pad 17: GND -> /GND
- J5 pad 30: GND -> /GND
- J5 pad 6: GND -> /GND
- J6 pad 1: GND -> /GND
- J6 pad 17: GND -> /GND
- J6 pad 23: GND -> /GND
- J6 pad 30: GND -> /GND
- J6 pad 8: GND -> /GND
- TP30 pad 1: GND -> /GND
Routing:
- net GND: track 8.90 -> 8.26 mm
- net /GND: track 0.00 -> 0.65 mm

Commit message: 1219
Parts:
- removed G***: LOGO, MyLibrary:kamo20
- J1, J2: footprint samacsys:DF40C60DS04V51 -> SamacSys_Parts:DF40C60DS04V51; moved to F.Cu
- moved REF** 29.4 mm to (109.2, 99.1)
- moved REF** 29.4 mm to (109.2, 109.2)
- moved REF** 29.4 mm to (119.4, 101.6)
- moved REF** 29.4 mm to (116.8, 101.6)
- moved REF** 29.4 mm to (119.4, 104.1)
- moved REF** 29.4 mm to (109.2, 104.1)
- moved REF** 29.4 mm to (109.2, 101.6)
- moved REF** 29.4 mm to (116.8, 99.1)
- moved REF** 29.4 mm to (109.2, 106.7)
- moved REF** 29.4 mm to (116.8, 104.1)
- moved REF** 29.4 mm to (111.8, 104.1)
- moved REF** 29.4 mm to (114.3, 106.7)
- moved REF** 29.4 mm to (111.8, 101.6)
- moved REF** 29.4 mm to (111.8, 106.7)
- moved REF** 29.4 mm to (111.8, 99.1)
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Routing:
- net /VDD_1V8: track 83.1 -> 13.5 mm, vias 1 -> 0
- net +2V5: track 70.8 -> 13.5 mm, vias 1 -> 0
- net /IOB91A: track 62.0 -> 9.18 mm, vias 1 -> 0
- net /IOB4A: track 58.2 -> 8.25 mm
- net /IOB91B: track 57.0 -> 8.68 mm, vias 1 -> 0
- net /IOT31A: track 56.8 -> 8.50 mm
- net /IOL12A: track 55.6 -> 8.50 mm
- net /IOT56A: track 55.1 -> 8.55 mm
- net /IOB26A: track 54.2 -> 8.25 mm
- net /IOL5A: track 53.8 -> 8.50 mm
- net /M0_D0P: track 53.6 -> 8.25 mm
- net /IOT58A: track 53.2 -> 8.50 mm
- net /IOB4B: track 53.0 -> 8.29 mm
- net /IOL12B: track 52.2 -> 8.00 mm
- net /IOL9A: track 52.1 -> 8.50 mm
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Other:
- copper layers 2 -> 4

Commit message: 1219
Parts:
- moved TP69 70.0 mm to (137.3, 146.7)
- moved TP70 69.9 mm to (137.3, 122.6)
- moved TP123 67.5 mm to (206.0, 150.5)
- moved TP124 67.4 mm to (205.9, 126.5)
- moved TP71 64.9 mm to (139.8, 150.5)
- moved TP72 64.8 mm to (139.8, 126.4)
- moved TP122 62.3 mm to (203.3, 122.6)
- moved TP121 62.3 mm to (203.3, 146.7)
- moved TP73 60.0 mm to (142.4, 146.7)
- moved TP74 59.8 mm to (142.4, 122.6)
- moved TP120 57.3 mm to (200.8, 126.5)
- moved TP119 57.2 mm to (200.8, 150.5)
- moved TP75 54.8 mm to (144.9, 150.5)
- moved TP76 54.7 mm to (144.9, 126.4)
- moved TP117 52.1 mm to (198.2, 146.7)
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Routing:
- net /VCCIO0/1: track 13.8 -> 0.00 mm
- net /VCCIO6/7: track 12.9 -> 0.00 mm
- net /IOT72A: track 12.7 -> 0.00 mm
- net /IOT68A: track 12.7 -> 0.00 mm
- net /IOT66A: track 12.7 -> 0.00 mm
- net /IOT63A: track 12.7 -> 0.00 mm
- net /IOT61A: track 12.7 -> 0.00 mm
- net /IOT23A: track 9.39 -> 0.00 mm
- net /IOT21A: track 9.39 -> 0.00 mm
- net /IOT19A: track 9.39 -> 0.00 mm
- net /IOT15A: track 9.39 -> 0.00 mm
- net /IOT11A: track 9.39 -> 0.00 mm
- net /IOL3B: track 9.39 -> 0.00 mm
- net /IOL14B: track 9.39 -> 0.00 mm
- net /IOT56A: track 8.55 -> 0.00 mm
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
Commit message: 1220
Parts:
- removed the REF** at (213.8, 101.2)
- removed the REF** at (213.8, 107.3)
- added J7: Conn_01x05, Connector_PinSocket_2.54mm:PinSocket_1x05_P2.54mm_Vertical, F.Cu at (218.2, 101.0)
- J3: value Conn_01x30 -> Conn_01x18; footprint Connector_PinHeader_2.54mm:PinHeader_1x30_P2.54mm_Vertical_SMD_Pin1Left -> Connector_PinHeader_2.54mm:PinHeader_1x18_P2.54mm_Vertical_SMD_Pin1Left
- TP11, TP12, TP14, TP15, TP17, TP18, TP19, TP2, TP20, TP22, TP23, TP24, TP25, TP26, TP27, TP28, TP29, TP3, TP30, TP5, TP6, TP8, TP9: footprint TestPoint:TestPoint_THTPad_1.5x1.5mm_Drill0.7mm -> TestPoint:TestPoint_Pad_1.5x1.5mm
- TP35, TP37, TP40, TP42, TP43, TP44, TP45, TP46, TP47, TP48, TP49, TP50, TP51, TP52, TP53, TP54, TP55, TP56, TP57, TP58, TP60: footprint TestPoint:TestPoint_Pad_1.5x1.5mm -> TestPoint:TestPoint_THTPad_1.5x1.5mm_Drill0.7mm
- moved TP42 39.0 mm to (213.7, 111.1)
- moved TP1 38.3 mm to (213.7, 101.0)
- moved TP40 33.3 mm to (213.7, 108.6)
- moved TP37 23.9 mm to (213.7, 106.0)
- moved TP44 23.5 mm to (175.4, 67.2)
- moved TP46 23.5 mm to (170.3, 67.2)
- moved TP48 23.5 mm to (165.2, 67.2)
- moved TP50 23.5 mm to (160.1, 67.2)
- moved TP52 23.5 mm to (155.1, 67.2)
- moved TP54 23.5 mm to (150.0, 67.2)
- moved TP56 23.5 mm to (144.9, 67.2)
- moved TP58 23.5 mm to (139.8, 67.2)
- moved TP60 23.5 mm to (134.7, 67.2)
- moved TP12 23.4 mm to (180.5, 89.7)
- moved TP14 23.4 mm to (175.4, 89.7)
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Connections:
- J1 pad 1: /GND -> GND
- J1 pad 15: /GND -> GND
- J1 pad 2: /GND -> GND
- J1 pad 27: /GND -> GND
- J1 pad 28: /GND -> GND
- J1 pad 45: /GND -> GND
- J1 pad 50: /GND -> GND
- J1 pad 59: /GND -> GND
- J1 pad 60: /GND -> GND
- J2 pad 1: /GND -> GND
- J2 pad 19: /GND -> GND
- J2 pad 29: /GND -> GND
- J2 pad 35: /GND -> GND
- J2 pad 41: /GND -> GND
- J2 pad 47: /GND -> GND
- J2 pad 53: /GND -> GND
- J2 pad 59: /GND -> GND
- J3 pad 1: +5V -> /IOB91B
- J3 pad 10: +2V5 -> /IOR24A
- J3 pad 11: /VDD_1V8 -> /IOR22B
- J3 pad 12: /VDD_1V8 -> /IOR22A
- J3 pad 13: /IOB91B -> /IOR20B
- J3 pad 14: /IOB91A -> /IOR20A
- J3 pad 15: /IOB89B -> /IOR18B
- J3 pad 16: /IOB89A -> /IOR18A
- J3 pad 17: /IOR33B -> /VCCIO2/3
- J3 pad 18: /IOR33A -> /VCCIO2/3
- J3 pad 2: +5V -> /IOB91A
- J3 pad 3: +5V -> /IOB89B
- J3 pad 4: +5V -> /IOB89A
- J3 pad 5: +5V -> /IOR33B
- J3 pad 6: +3V3 -> /IOR33A
- J3 pad 7: +3V3 -> /IOR31B
- J3 pad 8: +3V3 -> /IOR31A
- J3 pad 9: +2V5 -> /IOR24B
- J4 pad 1: /GND -> GND
- J4 pad 10: /GND -> GND
- J4 pad 13: /GND -> GND
- J4 pad 16: /GND -> GND
- J4 pad 21: /GND -> GND
- J4 pad 30: /GND -> GND
- J4 pad 4: /GND -> GND
- J4 pad 7: /GND -> GND
- J5 pad 1: /GND -> GND
- J5 pad 17: /GND -> GND
- J5 pad 30: /GND -> GND
- J5 pad 6: /GND -> GND
- J6 pad 1: /GND -> GND
- J6 pad 17: /GND -> GND
- J6 pad 23: /GND -> GND
- J6 pad 30: /GND -> GND
- J6 pad 8: /GND -> GND
- TP30 pad 1: /GND -> GND
Routing:
- net +5V: track 27.2 -> 0.00 mm
- net +3V3: track 20.8 -> 0.00 mm
- net /IOR18B: track 14.9 -> 0.00 mm
- net /VDD_1V8: track 13.5 -> 0.00 mm
- net /VCCIO2/3: track 13.5 -> 0.00 mm
- net +2V5: track 13.5 -> 0.00 mm
- net /IOR31A: track 9.18 -> 0.00 mm
- net /IOR24A: track 9.18 -> 0.00 mm
- net /IOR22A: track 9.18 -> 0.00 mm
- net /IOR20A: track 9.18 -> 0.00 mm
- net /IOB89A: track 9.18 -> 0.00 mm
- net /IOR33A: track 9.18 -> 0.00 mm
- net /IOR18A: track 9.18 -> 0.00 mm
- net /IOB91A: track 9.18 -> 0.00 mm
- net /IOR33B: track 8.68 -> 0.00 mm
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Other:
- copper layers 4 -> 2
