File: base_board1/base_board1.kicad_sch (KiCad schematic)
At the start: 123 parts, among them J1 DF40C-60DP-0.4V_51_, J2 DF40C-60DP-0.4V_51_, J3 Conn_01x30, J4 Conn_01x30, J5 Conn_01x30, J6 Conn_01x30

Commit message: 1218
Parts:
- removed TP1, TP10, TP13, TP16, TP21, TP4, TP61, TP63, TP7: TestPoint, TestPoint:TestPoint_THTPad_1.5x1.5mm_Drill0.7mm, symbol Connector:TestPoint
- removed TP111, TP116, TP125, TP126, TP127, TP128, TP62, TP64, TP65, TP66, TP67, TP68, TP81, TP93, TP94: TestPoint, TestPoint:TestPoint_Pad_1.5x1.5mm, symbol Connector:TestPoint

Commit message: 1218
Parts:
- removed J1, J2: DF40C-60DP-0.4V_51_, SamacSys_Parts:DF40C-60DP-0.4V_51_, symbol samacsys:DF40C-60DP-0.4V_51_
- added J1, J2: DF40C-60DS-0.4V_51_, DF40C60DS04V51, symbol samacsys:DF40C-60DS-0.4V_51_
Connections:
- net +2V5: now also J2.41, J2.43
- net +3V3: now also J2.45, J2.47, J2.49
- net +5V: now also J2.51, J2.53, J2.55, J2.57, J2.59
- net DONE: now also J1.26
- net GND: now also J1.1, J1.16, J1.2, J1.27, J1.28, J1.46, J1.49, J1.59, J1.60, J2.2, J2.20, J2.30, J2.36, J2.42, J2.48, J2.54, J2.60
- net IOB12B: now also J2.16
- net IOB14B: now also J2.18
- net IOB24A: now also J2.12
- net IOB26A: now also J2.8
- net IOB26B: now also J2.10
- net IOB4A: now also J2.4
- net IOB4B: now also J2.6
- net IOB56A: now also J1.20
- net IOB56B: now also J1.22
- net IOB60A: now also J1.24
- net IOB89A: now also J2.29
- net IOB89B: now also J2.31
- net IOB91A: now also J2.33
- net IOB91B: now also J2.35
- net IOL12A: now also J1.56
- net IOL12B: now also J1.58
- net IOL14A: now also J1.55
- net IOL14B: now also J1.57
- net IOL3A: now also J1.51
- net IOL3B: now also J1.53
- net IOL5A: now also J1.52
- net IOL5B: now also J1.54
- net IOL9A: now also J1.48
- net IOL9B: now also J1.50
- net IOR18A: now also J2.5
- net IOR18B: now also J2.7
- net IOR20A: now also J2.9
- net IOR20B: now also J2.11
- net IOR22A: now also J2.13
- net IOR22B: now also J2.15
- net IOR24A: now also J2.17
- net IOR24B: now also J2.19
- net IOR31A: now also J2.21
- net IOR31B: now also J2.23
- net IOR33A: now also J2.25
- net IOR33B: now also J2.27
- net IOT11A: now also J1.45
- net IOT11B: now also J1.47
- net IOT15A: now also J1.41
- net IOT15B: now also J1.43
- net IOT19A: now also J1.37
- net IOT19B: now also J1.39
- net IOT1A: now also J1.34
- net IOT1B: now also J1.36
- net IOT21A: now also J1.33
- net IOT21B: now also J1.35
- net IOT23A: now also J1.29
- net IOT23B: now also J1.31
- net IOT31A: now also J1.4
- net IOT31B: now also J1.6
- net IOT3A: now also J1.38
- net IOT3B: now also J1.40
- net IOT56A: now also J1.8
- net IOT56B: now also J1.10
- net IOT58A: now also J1.12
- net IOT58B: now also J1.14
- net IOT61A: now also J1.3
- net IOT61B: now also J1.5
- net IOT63A: now also J1.7
- net IOT63B: now also J1.9
- net IOT66A: now also J1.11
- net IOT66B: now also J1.13
- net IOT68A: now also J1.15
- net IOT68B: now also J1.17
- net IOT72A: now also J1.19
- net IOT72B: now also J1.21
- net IOT7A: now also J1.42
- net IOT7B: now also J1.44
- net M0_CKN: now also J2.46
- net M0_CKP: now also J2.44
- net M0_D0N: now also J2.58
- net M0_D0P: now also J2.56
- net M0_D1N: now also J2.52
- net M0_D1P: now also J2.50
- net M0_D2N: now also J2.40
- net M0_D2P: now also J2.38
- net M0_D3N: now also J2.34
- net M0_D3P: now also J2.32
- net READY: now also J1.18
- net RECONFIG: now also J2.14
- net TCK: now also J2.22
- net TDI: now also J2.28
- net TDO: now also J2.26
- net TMS: now also J2.24
- net VCCIO0/1: now also J1.23, J1.25
- net VCCIO2/3: now also J2.1, J2.3
- net VCCIO6/7: now also J1.30, J1.32
- net VDD_1V8: now also J2.37, J2.39

Commit message: 1219
Parts:
- removed J1, J2: DF40C-60DS-0.4V_51_, DF40C60DS04V51, symbol samacsys:DF40C-60DS-0.4V_51_
- added J1, J2: DF40C-60DS-0.4V_51_, SamacSys_Parts:DF40C60DS04V51, symbol SamacSys_Parts:DF40C-60DS-0.4V_51_
Connections:
- net +2V5: now also J2.42, J2.44
- net +3V3: now also J2.46, J2.48, J2.50
- net +5V: now also J2.52, J2.54, J2.56, J2.58, J2.60
- net DONE: now also J1.25
- net GND: now also J1.1, J1.15, J1.2, J1.27, J1.28, J1.45, J1.50, J1.59, J1.60, J2.1, J2.19, J2.29, J2.35, J2.41, J2.47, J2.53, J2.59
- net IOB12B: now also J2.15
- net IOB14B: now also J2.17
- net IOB24A: now also J2.11
- net IOB26A: now also J2.7
- net IOB26B: now also J2.9
- net IOB4A: now also J2.3
- net IOB4B: now also J2.5
- net IOB56A: now also J1.19
- net IOB56B: now also J1.21
- net IOB60A: now also J1.23
- net IOB89A: now also J2.30
- net IOB89B: now also J2.32
- net IOB91A: now also J2.34
- net IOB91B: now also J2.36
- net IOL12A: now also J1.55
- net IOL12B: now also J1.57
- net IOL14A: now also J1.56
- net IOL14B: now also J1.58
- net IOL3A: now also J1.52
- net IOL3B: now also J1.54
- net IOL5A: now also J1.51
- net IOL5B: now also J1.53
- net IOL9A: now also J1.47
- net IOL9B: now also J1.49
- net IOR18A: now also J2.6
- net IOR18B: now also J2.8
- net IOR20A: now also J2.10
- net IOR20B: now also J2.12
- net IOR22A: now also J2.14
- net IOR22B: now also J2.16
- net IOR24A: now also J2.18
- net IOR24B: now also J2.20
- net IOR31A: now also J2.22
- net IOR31B: now also J2.24
- net IOR33A: now also J2.26
- net IOR33B: now also J2.28
- net IOT11A: now also J1.46
- net IOT11B: now also J1.48
- net IOT15A: now also J1.42
- net IOT15B: now also J1.44
- net IOT19A: now also J1.38
- net IOT19B: now also J1.40
- net IOT1A: now also J1.33
- net IOT1B: now also J1.35
- net IOT21A: now also J1.34
- net IOT21B: now also J1.36
- net IOT23A: now also J1.30
- net IOT23B: now also J1.32
- net IOT31A: now also J1.3
- net IOT31B: now also J1.5
- net IOT3A: now also J1.37
- net IOT3B: now also J1.39
- net IOT56A: now also J1.7
- net IOT56B: now also J1.9
- net IOT58A: now also J1.11
- net IOT58B: now also J1.13
- net IOT61A: now also J1.4
- net IOT61B: now also J1.6
- net IOT63A: now also J1.8
- net IOT63B: now also J1.10
- net IOT66A: now also J1.12
- net IOT66B: now also J1.14
- net IOT68A: now also J1.16
- net IOT68B: now also J1.18
- net IOT72A: now also J1.20
- net IOT72B: now also J1.22
- net IOT7A: now also J1.41
- net IOT7B: now also J1.43
- net M0_CKN: now also J2.45
- net M0_CKP: now also J2.43
- net M0_D0N: now also J2.57
- net M0_D0P: now also J2.55
- net M0_D1N: now also J2.51
- net M0_D1P: now also J2.49
- net M0_D2N: now also J2.39
- net M0_D2P: now also J2.37
- net M0_D3N: now also J2.33
- net M0_D3P: now also J2.31
- net READY: now also J1.17
- net RECONFIG: now also J2.13
- net TCK: now also J2.21
- net TDI: now also J2.27
- net TDO: now also J2.25
- net TMS: now also J2.23
- net VCCIO0/1: now also J1.24, J1.26
- net VCCIO2/3: now also J2.2, J2.4
- net VCCIO6/7: now also J1.29, J1.31
- net VDD_1V8: now also J2.38, J2.40

Commit message: 1220
Parts:
- removed J3: Conn_01x30, Connector_PinHeader_2.54mm:PinHeader_1x30_P2.54mm_Vertical_SMD_Pin1Left, symbol Connector_Generic:Conn_01x30
- added J3: Conn_01x18, Connector_PinHeader_2.54mm:PinHeader_1x18_P2.54mm_Vertical_SMD_Pin1Left, symbol Connector_Generic:Conn_01x18
- added J7: Conn_01x05, Connector_PinSocket_2.54mm:PinSocket_1x05_P2.54mm_Vertical, symbol Connector_Generic:Conn_01x05
- TP101, TP103, TP105, TP107, TP109, TP113, TP115, TP117, TP119, TP121, TP123, TP35, TP37, TP40, TP42, TP43, TP44, TP45, TP46, TP47, TP48, TP49, TP50, TP51, TP52, TP53, TP54, TP55, TP56, TP57, TP58, TP60, TP69, TP71, TP73, TP75, TP77, TP79, TP83, TP85, TP87, TP89, TP91, TP95, TP99: footprint TestPoint:TestPoint_Pad_1.5x1.5mm -> TestPoint:TestPoint_THTPad_1.5x1.5mm_Drill0.7mm
- TP11, TP12, TP14, TP15, TP17, TP18, TP19, TP2, TP20, TP22, TP23, TP24, TP25, TP26, TP27, TP28, TP29, TP3, TP30, TP5, TP6, TP8, TP9: footprint TestPoint:TestPoint_THTPad_1.5x1.5mm_Drill0.7mm -> TestPoint:TestPoint_Pad_1.5x1.5mm
Connections:
- net +2V5: now also J7.4 (Pin_4)
- net +3V3: now also J7.3 (Pin_3)
- net +5V: now also J7.2 (Pin_2)
- net GND: now also J7.1 (Pin_1)
- net IOB89A: now also J3.4 (Pin_4)
- net IOB89B: now also J3.3 (Pin_3)
- net IOB91A: now also J3.2 (Pin_2)
- net IOB91B: now also J3.1 (Pin_1)
- net IOR18A: now also J3.16 (Pin_16)
- net IOR18B: now also J3.15 (Pin_15)
- net IOR20A: now also J3.14 (Pin_14)
- net IOR20B: now also J3.13 (Pin_13)
- net IOR22A: now also J3.12 (Pin_12)
- net IOR22B: now also J3.11 (Pin_11)
- net IOR24A: now also J3.10 (Pin_10)
- net IOR24B: now also J3.9 (Pin_9)
- net IOR31A: now also J3.8 (Pin_8)
- net IOR31B: now also J3.7 (Pin_7)
- net IOR33A: now also J3.6 (Pin_6)
- net IOR33B: now also J3.5 (Pin_5)
- net VCCIO2/3: now also J3.17 (Pin_17), J3.18 (Pin_18)
- net VDD_1V8: now also J7.5 (Pin_5)
