File: ds_test_board_v3/ds_test_board3/ds_test_board3.kicad_sch (KiCad schematic)
At the start: 125 parts, among them J1 DF40C-60DP-0.4V_51_, J2 DF40C-60DP-0.4V_51_, J3 Conn_01x30, J4 Conn_01x30, J5 Conn_01x30, J6 Conn_01x30

Commit message: 1205
Parts:
- removed TP90, TP97: TestPoint, TestPoint:TestPoint_Pad_1.5x1.5mm, symbol Connector:TestPoint
Connections:
- net +2V5: no longer J1.46, J5.8 (Pin_8), TP112.1
- net +3V3: no longer J1.48, J5.7 (Pin_7), TP114.1
- net +5V: no longer J1.52, J1.54, J1.56, J1.58, J5.2 (Pin_2), J5.3 (Pin_3), J5.4 (Pin_4), J5.5 (Pin_5), TP118.1, TP120.1, TP122.1, TP124.1
- net GND: now also J1.15, J1.2, J1.27, J1.28, J1.45, J1.50, J1.60, J5.1 (Pin_1), J5.17 (Pin_17), J5.30 (Pin_30), J5.6 (Pin_6), J6.17 (Pin_17), J6.23 (Pin_23), J6.8 (Pin_8), TP111.1, TP116.1, TP126.1, TP68.1, TP81.1, TP93.1, TP94.1; no longer J1.19, J1.29, J1.35, J1.41, J1.47, J1.53, J6.10 (Pin_10), J6.13 (Pin_13), J6.16 (Pin_16), J6.21 (Pin_21), J6.4 (Pin_4), J6.7 (Pin_7), TP101.1, TP107.1, TP113.1, TP119.1, TP85.1, TP95.1
- net IOB12B: no longer J1.15, J6.23 (Pin_23), TP81.1
- net IOB14B: no longer J1.17, J6.22 (Pin_22), TP83.1
- net IOB24A: no longer J1.11, J6.25 (Pin_25), TP77.1
- net IOB26A: no longer J1.7, J6.27 (Pin_27), TP73.1
- net IOB26B: no longer J1.9, J6.26 (Pin_26), TP75.1
- net IOB4A: no longer J1.3, J6.29 (Pin_29), TP69.1
- net IOB4B: no longer J1.5, J6.28 (Pin_28), TP71.1
- net IOB89A: no longer J1.30, J5.16 (Pin_16), TP96.1
- net IOB89B: no longer J1.32, J5.15 (Pin_15), TP98.1
- net IOB91A: no longer J1.34, J5.14 (Pin_14), TP100.1
- net IOB91B: no longer J1.36, J5.13 (Pin_13), TP102.1
- net IOR18A: no longer J1.6, J5.28 (Pin_28), TP72.1
- net IOR18B: no longer J1.8, J5.27 (Pin_27), TP74.1
- net IOR20A: no longer J1.10, J5.26 (Pin_26), TP76.1
- net IOR20B: no longer J1.12, J5.25 (Pin_25), TP78.1
- net IOR22A: no longer J1.14, J5.24 (Pin_24), TP80.1
- net IOR22B: no longer J1.16, J5.23 (Pin_23), TP82.1
- net IOR24A: no longer J1.18, J5.22 (Pin_22), TP84.1
- net IOR24B: no longer J1.20, J5.21 (Pin_21), TP86.1
- net IOR31A: no longer J1.22, J5.20 (Pin_20), TP88.1
- net IOR31B: no longer J1.24, J5.19 (Pin_19)
- net IOR33A: no longer J1.26, J5.18 (Pin_18), TP92.1
- net IOR33B: no longer J1.28, J5.17 (Pin_17), TP94.1
- net M0_CKN: no longer J1.45, J6.8 (Pin_8), TP111.1
- net M0_CKP: no longer J1.43, J6.9 (Pin_9), TP109.1
- net M0_D0N: no longer J1.57, J6.2 (Pin_2), TP123.1
- net M0_D0P: no longer J1.55, J6.3 (Pin_3), TP121.1
- net M0_D1N: no longer J1.51, J6.5 (Pin_5), TP117.1
- net M0_D1P: no longer J1.49, J6.6 (Pin_6), TP115.1
- net M0_D2N: no longer J1.39, J6.11 (Pin_11), TP105.1
- net M0_D2P: no longer J1.37, J6.12 (Pin_12), TP103.1
- net M0_D3N: no longer J1.33, J6.14 (Pin_14), TP99.1
- net M0_D3P: no longer J1.31, J6.15 (Pin_15)
- net RECONFIG: no longer J1.13, J6.24 (Pin_24), TP79.1
- net TCK: no longer J1.21, J6.20 (Pin_20), TP87.1
- net TDI: no longer J1.27, J6.17 (Pin_17), TP93.1
- net TDO: no longer J1.25, J6.18 (Pin_18), TP91.1
- net TMS: no longer J1.23, J6.19 (Pin_19), TP89.1
- net VCCIO2/3: no longer J1.2, J5.30 (Pin_30), TP68.1
- net VDD_1V8: no longer J1.38, J1.40, J5.11 (Pin_11), J5.12 (Pin_12), TP104.1, TP106.1
- net IOT61A: now reaches J1.4, J5.29 (Pin_29), TP70.1
- net IOT15A: now reaches J1.42, J5.10 (Pin_10), TP108.1
- net IOT15B: now reaches J1.44, J5.9 (Pin_9), TP110.1
- new net DONE: J1.25, J6.18 (Pin_18), TP91.1
- new net IOB56A: J1.19, J6.21 (Pin_21), TP85.1
- new net IOB56B: J1.21, J6.20 (Pin_20), TP87.1
- new net IOB60A: J1.23, J6.19 (Pin_19), TP89.1
- new net IOL12A: J1.55, J6.3 (Pin_3), TP121.1
- new net IOL12B: J1.57, J6.2 (Pin_2), TP123.1
- new net IOL14A: J1.56, J5.3 (Pin_3), TP122.1
- new net IOL14B: J1.58, J5.2 (Pin_2), TP124.1
- new net IOL3A: J1.52, J5.5 (Pin_5), TP118.1
- new net IOL3B: J1.54, J5.4 (Pin_4), TP120.1
- new net IOL5A: J1.51, J6.5 (Pin_5), TP117.1
- new net IOL5B: J1.53, J6.4 (Pin_4), TP119.1
- new net IOL9A: J1.47, J6.7 (Pin_7), TP113.1
- new net IOL9B: J1.49, J6.6 (Pin_6), TP115.1
- new net IOT11A: J1.46, J5.8 (Pin_8), TP112.1
- new net IOT11B: J1.48, J5.7 (Pin_7), TP114.1
- new net IOT19A: J1.38, J5.12 (Pin_12), TP104.1
- new net IOT19B: J1.40, J5.11 (Pin_11), TP106.1
- new net IOT1A: J1.33, J6.14 (Pin_14), TP99.1
- new net IOT1B: J1.35, J6.13 (Pin_13), TP101.1
- new net IOT21A: J1.34, J5.14 (Pin_14), TP100.1
- new net IOT21B: J1.36, J5.13 (Pin_13), TP102.1
- new net IOT23A: J1.30, J5.16 (Pin_16), TP96.1
- new net IOT23B: J1.32, J5.15 (Pin_15), TP98.1
- new net IOT31A: J1.3, J6.29 (Pin_29), TP69.1
- new net IOT31B: J1.5, J6.28 (Pin_28), TP71.1
- new net IOT3A: J1.37, J6.12 (Pin_12), TP103.1
- new net IOT3B: J1.39, J6.11 (Pin_11), TP105.1
- new net IOT56A: J1.7, J6.27 (Pin_27), TP73.1
- new net IOT56B: J1.9, J6.26 (Pin_26), TP75.1
- new net IOT58A: J1.11, J6.25 (Pin_25), TP77.1
- new net IOT58B: J1.13, J6.24 (Pin_24), TP79.1
- new net IOT61B: J1.6, J5.28 (Pin_28), TP72.1
- new net IOT63A: J1.8, J5.27 (Pin_27), TP74.1
- new net IOT63B: J1.10, J5.26 (Pin_26), TP76.1
- new net IOT66A: J1.12, J5.25 (Pin_25), TP78.1
- new net IOT66B: J1.14, J5.24 (Pin_24), TP80.1
- new net IOT68A: J1.16, J5.23 (Pin_23), TP82.1
- new net IOT68B: J1.18, J5.22 (Pin_22), TP84.1
- new net IOT72A: J1.20, J5.21 (Pin_21), TP86.1
- new net IOT72B: J1.22, J5.20 (Pin_20), TP88.1
- new net IOT7A: J1.41, J6.10 (Pin_10), TP107.1
- new net IOT7B: J1.43, J6.9 (Pin_9), TP109.1
- new net READY: J1.17, J6.22 (Pin_22), TP83.1
- new net VCCIO0/1: J1.24, J1.26, J5.18 (Pin_18), J5.19 (Pin_19), TP92.1
- new net VCCIO6/7: J1.29, J1.31, J6.15 (Pin_15), J6.16 (Pin_16), TP95.1
Other:
- note added: "Upper Connector"
