File: ds_test_board_v3/ds_test_board3/ds_test_board3.kicad_pcb (KiCad board)
At the start: 2 copper layers, 91.4 x 100 mm, 129 parts, among them J1 DF40C-60DP-0.4V_51_, J2 DF40C-60DP-0.4V_51_, J3 Conn_01x30, J4 Conn_01x30, J5 Conn_01x30, J6 Conn_01x30

Commit message: 1205
Parts:
- removed TP90, TP97: TestPoint, TestPoint:TestPoint_Pad_1.5x1.5mm
- J1: moved to B.Cu
- moved TP68 223.3 mm to (295.9, 154.9)
- moved TP67 134.5 mm to (205.7, 149.9)
- moved TP70 132.7 mm to (206.6, 109.3), turned to 180 degrees
- moved TP69 131.3 mm to (203.2, 153.7), turned to 180 degrees
- moved TP72 130.9 mm to (203.6, 109.3), turned to 180 degrees
- moved TP73 127.1 mm to (198.2, 153.7), turned to 180 degrees
- moved TP71 126.8 mm to (200.7, 149.9), turned to 180 degrees
- moved TP74 121.8 mm to (200.5, 109.3), turned to 180 degrees
- moved TP75 121.2 mm to (195.6, 149.9), turned to 180 degrees
- moved TP76 119.3 mm to (197.5, 109.3), turned to 180 degrees
- moved TP77 117.9 mm to (193.0, 153.7), turned to 180 degrees
- moved TP78 117.2 mm to (194.4, 109.3), turned to 180 degrees
- moved TP80 115.5 mm to (191.4, 109.3), turned to 180 degrees
- moved TP81 114.2 mm to (188.0, 153.7)
- moved TP79 113.2 mm to (190.5, 149.9), turned to 180 degrees
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Connections:
- net Net-(J5-Pin_10) renamed /IOT15A
- net Net-(J5-Pin_29) renamed /IOT61A
- net Net-(J5-Pin_9) renamed /IOT15B
- J1 pad 10: /IOR20A -> /IOT63B
- J1 pad 11: /IOB24A -> /IOT58A
- J1 pad 12: /IOR20B -> /IOT66A
- J1 pad 13: /RECONFIG -> /IOT58B
- J1 pad 14: /IOR22A -> /IOT66B
- J1 pad 15: /IOB12B -> GND
- J1 pad 16: /IOR22B -> /IOT68A
- J1 pad 17: /IOB14B -> /READY
- J1 pad 18: /IOR24A -> /IOT68B
- J1 pad 19: GND -> /IOB56A
- J1 pad 2: /VCCIO2/3 -> GND
- J1 pad 20: /IOR24B -> /IOT72A
- J1 pad 21: /TCK -> /IOB56B
- J1 pad 22: /IOR31A -> /IOT72B
- J1 pad 23: /TMS -> /IOB60A
- J1 pad 24: /IOR31B -> /VCCIO0/1
- J1 pad 25: /TDO -> /DONE
- J1 pad 26: /IOR33A -> /VCCIO0/1
- J1 pad 27: /TDI -> GND
- J1 pad 28: /IOR33B -> GND
- J1 pad 29: GND -> /VCCIO6/7
- J1 pad 3: /IOB4A -> /IOT31A
- J1 pad 30: /IOB89A -> /IOT23A
- J1 pad 31: /M0_D3P -> /VCCIO6/7
- J1 pad 32: /IOB89B -> /IOT23B
- J1 pad 33: /M0_D3N -> /IOT1A
- J1 pad 34: /IOB91A -> /IOT21A
- J1 pad 35: GND -> /IOT1B
- J1 pad 36: /IOB91B -> /IOT21B
- J1 pad 37: /M0_D2P -> /IOT3A
- J1 pad 38: /VDD_1V8 -> /IOT19A
- J1 pad 39: /M0_D2N -> /IOT3B
- J1 pad 40: /VDD_1V8 -> /IOT19B
- J1 pad 41: GND -> /IOT7A
- J1 pad 43: /M0_CKP -> /IOT7B
- J1 pad 45: /M0_CKN -> GND
- J1 pad 46: +2V5 -> /IOT11A
- J1 pad 47: GND -> /IOL9A
- J1 pad 48: +3V3 -> /IOT11B
- J1 pad 49: /M0_D1P -> /IOL9B
- J1 pad 5: /IOB4B -> /IOT31B
- J1 pad 50: Net-(J5-Pin_6) -> GND
- J1 pad 51: /M0_D1N -> /IOL5A
- J1 pad 52: +5V -> /IOL3A
- J1 pad 53: GND -> /IOL5B
- J1 pad 54: +5V -> /IOL3B
- J1 pad 55: /M0_D0P -> /IOL12A
- J1 pad 56: +5V -> /IOL14A
- J1 pad 57: /M0_D0N -> /IOL12B
- J1 pad 58: +5V -> /IOL14B
- J1 pad 6: /IOR18A -> /IOT61B
- J1 pad 60: Net-(J5-Pin_1) -> GND
- J1 pad 7: /IOB26A -> /IOT56A
- J1 pad 8: /IOR18B -> /IOT63A
- J1 pad 9: /IOB26B -> /IOT56B
- J5 pad 1: Net-(J5-Pin_1) -> GND
- J5 pad 11: /VDD_1V8 -> /IOT19B
- J5 pad 12: /VDD_1V8 -> /IOT19A
- J5 pad 13: /IOB91B -> /IOT21B
- J5 pad 14: /IOB91A -> /IOT21A
- J5 pad 15: /IOB89B -> /IOT23B
- J5 pad 16: /IOB89A -> /IOT23A
- J5 pad 17: /IOR33B -> GND
- J5 pad 18: /IOR33A -> /VCCIO0/1
- J5 pad 19: /IOR31B -> /VCCIO0/1
- J5 pad 2: +5V -> /IOL14B
- J5 pad 20: /IOR31A -> /IOT72B
- J5 pad 21: /IOR24B -> /IOT72A
- J5 pad 22: /IOR24A -> /IOT68B
- J5 pad 23: /IOR22B -> /IOT68A
- J5 pad 24: /IOR22A -> /IOT66B
- J5 pad 25: /IOR20B -> /IOT66A
- J5 pad 26: /IOR20A -> /IOT63B
- J5 pad 27: /IOR18B -> /IOT63A
- J5 pad 28: /IOR18A -> /IOT61B
- J5 pad 3: +5V -> /IOL14A
- J5 pad 30: /VCCIO2/3 -> GND
- J5 pad 4: +5V -> /IOL3B
- J5 pad 5: +5V -> /IOL3A
- J5 pad 6: Net-(J5-Pin_6) -> GND
- J5 pad 7: +3V3 -> /IOT11B
- J5 pad 8: +2V5 -> /IOT11A
- J6 pad 10: GND -> /IOT7A
- J6 pad 11: /M0_D2N -> /IOT3B
- J6 pad 12: /M0_D2P -> /IOT3A
- J6 pad 13: GND -> /IOT1B
- J6 pad 14: /M0_D3N -> /IOT1A
- J6 pad 15: /M0_D3P -> /VCCIO6/7
- J6 pad 16: GND -> /VCCIO6/7
- J6 pad 17: /TDI -> GND
- J6 pad 18: /TDO -> /DONE
- J6 pad 19: /TMS -> /IOB60A
- J6 pad 2: /M0_D0N -> /IOL12B
- J6 pad 20: /TCK -> /IOB56B
- J6 pad 21: GND -> /IOB56A
- J6 pad 22: /IOB14B -> /READY
- J6 pad 23: /IOB12B -> GND
- J6 pad 24: /RECONFIG -> /IOT58B
- J6 pad 25: /IOB24A -> /IOT58A
- J6 pad 26: /IOB26B -> /IOT56B
- J6 pad 27: /IOB26A -> /IOT56A
- J6 pad 28: /IOB4B -> /IOT31B
- J6 pad 29: /IOB4A -> /IOT31A
- J6 pad 3: /M0_D0P -> /IOL12A
- J6 pad 4: GND -> /IOL5B
- J6 pad 5: /M0_D1N -> /IOL5A
- J6 pad 6: /M0_D1P -> /IOL9B
- J6 pad 7: GND -> /IOL9A
- J6 pad 8: /M0_CKN -> GND
- J6 pad 9: /M0_CKP -> /IOT7B
- TP100 pad 1: /IOB91A -> /IOT21A
- TP101 pad 1: GND -> /IOT1B
- TP102 pad 1: /IOB91B -> /IOT21B
- TP103 pad 1: /M0_D2P -> /IOT3A
- TP104 pad 1: /VDD_1V8 -> /IOT19A
- TP105 pad 1: /M0_D2N -> /IOT3B
- TP106 pad 1: /VDD_1V8 -> /IOT19B
- TP107 pad 1: GND -> /IOT7A
- TP109 pad 1: /M0_CKP -> /IOT7B
- TP111 pad 1: /M0_CKN -> GND
- TP112 pad 1: +2V5 -> /IOT11A
- TP113 pad 1: GND -> /IOL9A
- TP114 pad 1: +3V3 -> /IOT11B
- TP115 pad 1: /M0_D1P -> /IOL9B
- TP116 pad 1: Net-(J5-Pin_6) -> GND
- TP117 pad 1: /M0_D1N -> /IOL5A
- TP118 pad 1: +5V -> /IOL3A
- TP119 pad 1: GND -> /IOL5B
- TP120 pad 1: +5V -> /IOL3B
- TP121 pad 1: /M0_D0P -> /IOL12A
- TP122 pad 1: +5V -> /IOL14A
- TP123 pad 1: /M0_D0N -> /IOL12B
- TP124 pad 1: +5V -> /IOL14B
- TP126 pad 1: Net-(J5-Pin_1) -> GND
- TP68 pad 1: /VCCIO2/3 -> GND
- TP69 pad 1: /IOB4A -> /IOT31A
- TP71 pad 1: /IOB4B -> /IOT31B
- TP72 pad 1: /IOR18A -> /IOT61B
- TP73 pad 1: /IOB26A -> /IOT56A
- TP74 pad 1: /IOR18B -> /IOT63A
- TP75 pad 1: /IOB26B -> /IOT56B
- TP76 pad 1: /IOR20A -> /IOT63B
- TP77 pad 1: /IOB24A -> /IOT58A
- TP78 pad 1: /IOR20B -> /IOT66A
- TP79 pad 1: /RECONFIG -> /IOT58B
- TP80 pad 1: /IOR22A -> /IOT66B
- TP81 pad 1: /IOB12B -> GND
- TP82 pad 1: /IOR22B -> /IOT68A
- TP83 pad 1: /IOB14B -> /READY
- TP84 pad 1: /IOR24A -> /IOT68B
- TP85 pad 1: GND -> /IOB56A
- TP86 pad 1: /IOR24B -> /IOT72A
- TP87 pad 1: /TCK -> /IOB56B
- TP88 pad 1: /IOR31A -> /IOT72B
- TP89 pad 1: /TMS -> /IOB60A
- TP91 pad 1: /TDO -> /DONE
- TP92 pad 1: /IOR33A -> /VCCIO0/1
- TP93 pad 1: /TDI -> GND
- TP94 pad 1: /IOR33B -> GND
- TP95 pad 1: GND -> /VCCIO6/7
- TP96 pad 1: /IOB89A -> /IOT23A
- TP98 pad 1: /IOB89B -> /IOT23B
- TP99 pad 1: /M0_D3N -> /IOT1A
Routing:
- net /VCCIO2/3: track 0.00 -> 54.5 mm, vias 0 -> 1
- net /IOR20B: track 0.00 -> 48.4 mm, vias 0 -> 1
- net /IOR18A: track 0.00 -> 48.1 mm, vias 0 -> 1
- net GND: track 523.0 -> 569.6 mm, vias 1 -> 2
- net /IOR22B: track 0.00 -> 46.4 mm, vias 0 -> 1
- net /IOR20A: track 0.00 -> 46.2 mm, vias 0 -> 1
- net /IOR18B: track 0.00 -> 45.1 mm, vias 0 -> 1
- net /IOR22A: track 0.00 -> 44.1 mm, vias 0 -> 1
- net /IOR24B: track 0.00 -> 44.0 mm, vias 0 -> 1
- net /IOR31B: track 0.00 -> 42.1 mm, vias 0 -> 1
- net /IOR24A: track 0.00 -> 41.8 mm, vias 0 -> 1
- net /IOR31A: track 0.00 -> 39.9 mm, vias 0 -> 1
- net /IOR33B: track 30.4 -> 38.6 mm
- net /IOR33A: track 28.3 -> 36.2 mm
- net /IOB89B: track 36.9 -> 38.4 mm
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Other:
- board text added: "+2V5"
- board text added: "+3V3"
- board text added: "+5V"
- board text added: "1V8"
- board text added: "Tang Primer 25K Tester Board"

Commit message: 1206
Parts:
- moved TP126 20.6 mm to (131.1, 129.0)
- moved TP118 20.3 mm to (142.2, 129.0)
- moved TP122 20.3 mm to (136.7, 129.0)
- moved TP114 20.1 mm to (147.3, 129.0)
- moved TP110 19.9 mm to (152.4, 129.0)
- moved TP72 19.9 mm to (200.7, 129.0)
- moved TP106 19.8 mm to (157.5, 129.0)
- moved TP76 19.8 mm to (195.6, 129.0)
- moved TP102 19.7 mm to (162.6, 129.0)
- moved TP88 19.7 mm to (180.3, 129.0)
- moved TP80 19.7 mm to (190.5, 129.0)
- moved TP92 19.7 mm to (175.3, 129.0)
- moved TP84 19.7 mm to (185.4, 129.0)
- moved TP98 19.7 mm to (167.6, 129.0)
- moved TP124 16.6 mm to (134.1, 125.0)
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Changed lines of the file:
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@@
   (net 97 "/IOL14B")
   (footprint "TestPoint:TestPoint_Pad_1.5x1.5mm" (layer "F.Cu")
-    (at 143.129 109.347 180)
+    (at 147.32 129.032 180)
     (descr "SMD rectangular pad as test Point, square 1.5mm side length")
     (tags "test point SMD pad rectangle square")
@@
   )
   (footprint "TestPoint:TestPoint_Pad_1.5x1.5mm" (layer "F.Cu")
-    (at 176.149 109.347 180)
+    (at 175.26 129.032 180)
     (descr "SMD rectangular pad as test Point, square 1.5mm side length")
     (tags "test point SMD pad rectangle square")
@@
   )
   (footprint "TestPoint:TestPoint_Pad_1.5x1.5mm" (layer "F.Cu")
-    (at 124.46 114.3 180)
+    (at 126.492 124.968 180)
     (descr "SMD rectangular pad as test Point, square 1.5mm side length")
     (tags "test point SMD pad rectangle square")
@@
   )
   (footprint "TestPoint:TestPoint_Pad_1.5x1.5mm" (layer "F.Cu")
-    (at 131.699 109.347 180)
+    (at 136.652 129.032 180)
     (descr "SMD rectangular pad as test Point, square 1.5mm side length")
     (tags "test point SMD pad rectangle square")
@@
   )
   (footprint "TestPoint:TestPoint_Pad_1.5x1.5mm" (layer "F.Cu")
-    (at 134.62 109.347 180)
+    (at 139.7 124.968 180)
     (descr "SMD rectangular pad as test Point, square 1.5mm side length")
     (tags "test point SMD pad rectangle square")
@@
   )
   (footprint "TestPoint:TestPoint_Pad_1.5x1.5mm" (layer "F.Cu")
-    (at 210.82 109.728)
+    (at 209.804 124.968)
     (descr "SMD rectangular pad as test Point, square 1.5mm side length")
     (tags "test point SMD pad rectangle square")
@@
   )
   (footprint "TestPoint:TestPoint_Pad_1.5x1.5mm" (layer "F.Cu")
-    (at 155.321 109.347 180)
+    (at 157.48 129.032 180)
     (descr "SMD rectangular pad as test Point, square 1.5mm side length")
     (tags "test point SMD pad rectangle square")
@@
   )
   (footprint "TestPoint:TestPoint_Pad_1.5x1.5mm" (layer "F.Cu")
-    (at 200.533 109.347 180)
+    (at 198.12 124.968 180)
     (descr "SMD rectangular pad as test Point, square 1.5mm side length")
     (tags "test point SMD pad rectangle square")
@@
   )
   (footprint "TestPoint:TestPoint_Pad_1.5x1.5mm" (layer "F.Cu")
-    (at 164.465 109.347 180)
+    (at 165.1 124.968 180)
     (descr "SMD rectangular pad as test Point, square 1.5mm side length")
     (tags "test point SMD pad rectangle square")
@@
   )
   (footprint "TestPoint:TestPoint_Pad_1.5x1.5mm" (layer "F.Cu")
-    (at 140.208 109.22)
+    (at 147.32 115.824)
     (descr "SMD rectangular pad as test Point, square 1.5mm side length")
     (tags "test point SMD pad rectangle square")
@@
   )
   (footprint "TestPoint:TestPoint_Pad_1.5x1.5mm" (layer "F.Cu")
-    (at 182.245 109.347 180)
+    (at 182.88 124.968 180)
     (descr "SMD rectangular pad as test Point, square 1.5mm side length")
     (tags "test point SMD pad rectangle square")
@@
   )
   (footprint "TestPoint:TestPoint_Pad_1.5x1.5mm" (layer "F.Cu")
-    (at 191.389 109.347 180)
+    (at 190.5 129.032 180)
     (descr "SMD rectangular pad as test Point, square 1.5mm side length")
     (tags "test point SMD pad rectangle square")
@@
   )
   (footprint "TestPoint:TestPoint_Pad_1.5x1.5mm" (layer "F.Cu")
-    (at 161.417 109.347 180)
+    (at 162.56 129.032 180)
     (descr "SMD rectangular pad as test Point, square 1.5mm side length")
     (tags "test point SMD pad rectangle square")
@@
   )
   (footprint "TestPoint:TestPoint_Pad_1.5x1.5mm" (layer "F.Cu")
-    (at 185.293 109.347 180)
+    (at 185.42 129.032 180)
     (descr "SMD rectangular pad as test Point, square 1.5mm side length")
     (tags "test point SMD pad rectangle square")
@@
   )
   (footprint "TestPoint:TestPoint_Pad_1.5x1.5mm" (layer "F.Cu")
-    (at 158.369 109.347 180)
+    (at 160.02 124.968 180)
     (descr "SMD rectangular pad as test Point, square 1.5mm side length")
     (tags "test point SMD pad rectangle square")
@@
   )
   (footprint "TestPoint:TestPoint_Pad_1.5x1.5mm" (layer "F.Cu")
-    (at 167.513 109.347 180)
+    (at 167.64 129.032 180)
     (descr "SMD rectangular pad as test Point, square 1.5mm side length")
     (tags "test point SMD pad rectangle square")
@@
   )
   (footprint "TestPoint:TestPoint_Pad_1.5x1.5mm" (layer "F.Cu")
-    (at 137.668 109.22 180)
+    (at 142.24 129.032 180)
     (descr "SMD rectangular pad as test Point, square 1.5mm side length")
     (tags "test point SMD pad rectangle square")
@@
   )
   (footprint "TestPoint:TestPoint_Pad_1.5x1.5mm" (layer "F.Cu")
-    (at 206.629 109.347 180)
+    (at 203.2 124.968 180)
     (descr "SMD rectangular pad as test Point, square 1.5mm side length")
     (tags "test point SMD pad rectangle square")
@@
   )
   (footprint "TestPoint:TestPoint_Pad_1.5x1.5mm" (layer "F.Cu")
-    (at 170.561 109.347 180)
+    (at 170.18 124.968 180)
     (descr "SMD rectangular pad as test Point, square 1.5mm side length")
     (tags "test point SMD pad rectangle square")
@@
   )
   (footprint "TestPoint:TestPoint_Pad_1.5x1.5mm" (layer "F.Cu")
-    (at 146.177 109.347 180)
+    (at 149.86 124.968 180)
     (descr "SMD rectangular pad as test Point, square 1.5mm side length")
     (tags "test point SMD pad rectangle square")
@@
   )
   (footprint "TestPoint:TestPoint_Pad_1.5x1.5mm" (layer "F.Cu")
-    (at 128.524 109.347 180)
+    (at 134.112 124.968 180)
     (descr "SMD rectangular pad as test Point, square 1.5mm side length")
     (tags "test point SMD pad rectangle square")
@@
   )
   (footprint "TestPoint:TestPoint_Pad_1.5x1.5mm" (layer "F.Cu")
-    (at 197.485 109.347 180)
+    (at 195.58 129.032 180)
     (descr "SMD rectangular pad as test Point, square 1.5mm side length")
     (tags "test point SMD pad rectangle square")
@@
   )
   (footprint "TestPoint:TestPoint_Pad_1.5x1.5mm" (layer "F.Cu")
-    (at 179.197 109.347 180)
+    (at 180.34 129.032 180)
     (descr "SMD rectangular pad as test Point, square 1.5mm side length")
     (tags "test point SMD pad rectangle square")
@@
   )
   (footprint "TestPoint:TestPoint_Pad_1.5x1.5mm" (layer "F.Cu")
-    (at 203.581 109.347 180)
+    (at 200.66 129.032 180)
     (descr "SMD rectangular pad as test Point, square 1.5mm side length")
     (tags "test point SMD pad rectangle square")
@@
   )
   (footprint "TestPoint:TestPoint_Pad_1.5x1.5mm" (layer "F.Cu")
-    (at 194.437 109.347 180)
+    (at 193.04 124.968 180)
     (descr "SMD rectangular pad as test Point, square 1.5mm side length")
     (tags "test point SMD pad rectangle square")
@@
   )
   (footprint "TestPoint:TestPoint_Pad_1.5x1.5mm" (layer "F.Cu")
-    (at 188.341 109.347 180)
+    (at 187.96 124.968 180)
     (descr "SMD rectangular pad as test Point, square 1.5mm side length")
     (tags "test point SMD pad rectangle square")
@@
   )
   (footprint "TestPoint:TestPoint_Pad_1.5x1.5mm" (layer "F.Cu")
-    (at 152.273 109.347 180)
+    (at 154.94 124.968 180)
     (descr "SMD rectangular pad as test Point, square 1.5mm side length")
     (tags "test point SMD pad rectangle square")
@@
   )
   (footprint "TestPoint:TestPoint_Pad_1.5x1.5mm" (layer "F.Cu")
-    (at 125.603 109.22 180)
+    (at 131.064 129.032 180)
     (descr "SMD rectangular pad as test Point, square 1.5mm side length")
     (tags "test point SMD pad rectangle square")
@@
   )
   (footprint "TestPoint:TestPoint_Pad_1.5x1.5mm" (layer "F.Cu")
-    (at 173.228 109.22)
+    (at 174.244 122.936)
     (descr "SMD rectangular pad as test Point, square 1.5mm side length")
     (tags "test point SMD pad rectangle square")
@@
   )
   (footprint "TestPoint:TestPoint_Pad_1.5x1.5mm" (layer "F.Cu")
-    (at 149.225 109.347 180)
+    (at 152.4 129.032 180)
     (descr "SMD rectangular pad as test Point, square 1.5mm side length")
     (tags "test point SMD pad rectangle square")

Commit message: 1211
Parts:
- TP101, TP103, TP105, TP107, TP109, TP111, TP113, TP115, TP117, TP119, TP121, TP123, TP125, TP128, TP66, TP67, TP69, TP71, TP73, TP75, TP77, TP79, TP81, TP83, TP85, TP87, TP89, TP91, TP93, TP95, TP99: footprint TestPoint:TestPoint_Pad_1.5x1.5mm -> TestPoint:TestPoint_THTPad_1.5x1.5mm_Drill0.7mm
- moved J1 8.18 mm to (168.6, 109.8)
- moved TP103 6.35 mm to (160.0, 143.5)
- moved TP107 6.35 mm to (154.9, 143.5)
- moved TP111 6.35 mm to (149.9, 143.5)
- moved TP115 6.35 mm to (144.8, 143.5)
- moved TP119 6.35 mm to (139.7, 143.5)
- moved TP123 6.35 mm to (134.6, 143.5)
- moved TP67 6.35 mm to (205.7, 143.5)
- moved TP71 6.35 mm to (200.7, 143.5)
- moved TP75 6.35 mm to (195.6, 143.5)
- moved TP79 6.35 mm to (190.5, 143.5)
- moved TP83 6.35 mm to (185.4, 143.5)
- moved TP87 6.35 mm to (180.3, 143.5)
- moved TP91 6.35 mm to (175.3, 143.5)
- moved TP99 6.35 mm to (165.1, 143.5)
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Routing:
- net GND: track 569.6 -> 824.8 mm
- net /IOT31A: track 0.00 -> 56.8 mm
- net /IOL12A: track 0.00 -> 55.6 mm
- net /IOT56A: track 0.00 -> 55.1 mm
- net /IOL5A: track 0.00 -> 53.8 mm
- net /IOT58A: track 0.00 -> 53.2 mm
- net /IOL12B: track 0.00 -> 52.2 mm
- net /IOL9A: track 0.00 -> 52.1 mm
- net /IOT31B: track 0.00 -> 51.6 mm
- net /IOL5B: track 0.00 -> 50.4 mm
- net /IOT7B: track 0.00 -> 50.3 mm
- net /IOT56B: track 0.00 -> 49.8 mm
- net /VCCIO6/7: track 0.00 -> 49.7 mm
- net /IOB56A: track 0.00 -> 49.7 mm
- net /IOL9B: track 0.00 -> 48.7 mm
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Other:
- board text added: "J1"
- board text added: "J2"

Commit message: 1215
Parts:
- moved TP126 1.02 mm to (132.1, 123.2)
- moved TP124 0.51 mm to (134.6, 118.7)
- moved TP122 0.46 mm to (137.1, 123.2)
Routing:
- net GND: track 824.8 -> 979.3 mm, vias 2 -> 5
- net /IOT61A: track 0.00 -> 52.7 mm, vias 0 -> 1
- net /IOT63A: track 0.00 -> 49.5 mm, vias 0 -> 1
- net /IOL14A: track 0.00 -> 48.9 mm, vias 0 -> 1
- net Net-(J1-Pad63): track 0.00 -> 48.2 mm
- net Net-(J1-Pad64): track 0.00 -> 48.1 mm, vias 0 -> 1
- net Net-(J1-Pad62): track 0.00 -> 47.1 mm
- net Net-(J1-Pad61): track 0.00 -> 47.0 mm, vias 0 -> 1
- net /IOT66A: track 0.00 -> 46.5 mm, vias 0 -> 1
- net /IOL14B: track 0.00 -> 45.7 mm, vias 0 -> 1
- net /IOL3A: track 0.00 -> 45.3 mm, vias 0 -> 1
- net /IOT63B: track 0.00 -> 44.5 mm, vias 0 -> 1
- net /IOT61B: track 0.00 -> 43.5 mm, vias 0 -> 1
- net /IOT68A: track 0.00 -> 42.3 mm, vias 0 -> 1
- net /IOL3B: track 0.00 -> 41.2 mm, vias 0 -> 1
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
Commit message: 1216
Parts:
- added G***: LOGO, MyLibrary:kamo20, F.Cu at (151.5, 112.5)
- added REF**: PinHeader_1x01_P2.54mm_Vertical, Connector_PinHeader_2.54mm:PinHeader_1x01_P2.54mm_Vertical, F.Cu at (137.2, 105.7)
- added REF**: PinHeader_1x01_P2.54mm_Vertical, Connector_PinHeader_2.54mm:PinHeader_1x01_P2.54mm_Vertical, F.Cu at (132.1, 103.1)
- added REF**: PinHeader_1x01_P2.54mm_Vertical, Connector_PinHeader_2.54mm:PinHeader_1x01_P2.54mm_Vertical, F.Cu at (124.5, 113.3)
- added REF**: PinHeader_1x01_P2.54mm_Vertical, Connector_PinHeader_2.54mm:PinHeader_1x01_P2.54mm_Vertical, F.Cu at (127.0, 108.2)
- added REF**: PinHeader_1x01_P2.54mm_Vertical, Connector_PinHeader_2.54mm:PinHeader_1x01_P2.54mm_Vertical, F.Cu at (124.5, 110.7)
- added REF**: PinHeader_1x01_P2.54mm_Vertical, Connector_PinHeader_2.54mm:PinHeader_1x01_P2.54mm_Vertical, F.Cu at (124.5, 100.6)
- added REF**: TestPoint_THTPad_2.0x2.0mm_Drill1.0mm, TestPoint:TestPoint_THTPad_2.0x2.0mm_Drill1.0mm, F.Cu at (209.8, 101.2)
- added REF**: PinHeader_1x01_P2.54mm_Vertical, Connector_PinHeader_2.54mm:PinHeader_1x01_P2.54mm_Vertical, F.Cu at (124.5, 115.8)
- added REF**: PinHeader_1x01_P2.54mm_Vertical, Connector_PinHeader_2.54mm:PinHeader_1x01_P2.54mm_Vertical, F.Cu at (132.1, 100.6)
- added REF**: PinHeader_1x01_P2.54mm_Vertical, Connector_PinHeader_2.54mm:PinHeader_1x01_P2.54mm_Vertical, F.Cu at (134.6, 100.6)
- added REF**: PinHeader_1x01_P2.54mm_Vertical, Connector_PinHeader_2.54mm:PinHeader_1x01_P2.54mm_Vertical, F.Cu at (127.0, 110.7)
- added REF**: PinHeader_1x01_P2.54mm_Vertical, Connector_PinHeader_2.54mm:PinHeader_1x01_P2.54mm_Vertical, F.Cu at (124.5, 95.5)
- added REF**: PinHeader_1x01_P2.54mm_Vertical, Connector_PinHeader_2.54mm:PinHeader_1x01_P2.54mm_Vertical, F.Cu at (127.0, 115.8)
- added REF**: PinHeader_1x01_P2.54mm_Vertical, Connector_PinHeader_2.54mm:PinHeader_1x01_P2.54mm_Vertical, F.Cu at (129.5, 108.2)
- added REF**: PinHeader_1x01_P2.54mm_Vertical, Connector_PinHeader_2.54mm:PinHeader_1x01_P2.54mm_Vertical, F.Cu at (139.7, 108.2)
- added REF**: PinHeader_1x01_P2.54mm_Vertical, Connector_PinHeader_2.54mm:PinHeader_1x01_P2.54mm_Vertical, F.Cu at (137.2, 103.1)
- added REF**: PinHeader_1x01_P2.54mm_Vertical, Connector_PinHeader_2.54mm:PinHeader_1x01_P2.54mm_Vertical, F.Cu at (124.5, 105.7)
- added REF**: TestPoint_THTPad_2.0x2.0mm_Drill1.0mm, TestPoint:TestPoint_THTPad_2.0x2.0mm_Drill1.0mm, F.Cu at (209.8, 107.3)
- added REF**: PinHeader_1x01_P2.54mm_Vertical, Connector_PinHeader_2.54mm:PinHeader_1x01_P2.54mm_Vertical, F.Cu at (134.6, 110.7)
- added REF**: SolderJumper-2_P1.3mm_Open_TrianglePad1.0x1.5mm, Jumper:SolderJumper-2_P1.3mm_Open_TrianglePad1.0x1.5mm, F.Cu at (128.5, 146.3)
- added REF**: PinHeader_1x01_P2.54mm_Vertical, Connector_PinHeader_2.54mm:PinHeader_1x01_P2.54mm_Vertical, F.Cu at (127.0, 98.0)
- added REF**: SolderJumper-2_P1.3mm_Open_TrianglePad1.0x1.5mm, Jumper:SolderJumper-2_P1.3mm_Open_TrianglePad1.0x1.5mm, F.Cu at (125.7, 79.2)
- added REF**: PinHeader_1x01_P2.54mm_Vertical, Connector_PinHeader_2.54mm:PinHeader_1x01_P2.54mm_Vertical, F.Cu at (144.8, 103.1)
- added REF**: PinHeader_1x01_P2.54mm_Vertical, Connector_PinHeader_2.54mm:PinHeader_1x01_P2.54mm_Vertical, F.Cu at (127.0, 103.1)
- added REF**: PinHeader_1x01_P2.54mm_Vertical, Connector_PinHeader_2.54mm:PinHeader_1x01_P2.54mm_Vertical, F.Cu at (132.1, 105.7)
- added REF**: PinHeader_1x01_P2.54mm_Vertical, Connector_PinHeader_2.54mm:PinHeader_1x01_P2.54mm_Vertical, F.Cu at (142.2, 103.1)
- added REF**: SolderJumper-2_P1.3mm_Open_TrianglePad1.0x1.5mm, Jumper:SolderJumper-2_P1.3mm_Open_TrianglePad1.0x1.5mm, F.Cu at (210.2, 134.6)
- added REF**: PinHeader_1x01_P2.54mm_Vertical, Connector_PinHeader_2.54mm:PinHeader_1x01_P2.54mm_Vertical, F.Cu at (124.5, 103.1)
- added REF**: PinHeader_1x01_P2.54mm_Vertical, Connector_PinHeader_2.54mm:PinHeader_1x01_P2.54mm_Vertical, F.Cu at (129.5, 105.7)
- added REF**: PinHeader_1x01_P2.54mm_Vertical, Connector_PinHeader_2.54mm:PinHeader_1x01_P2.54mm_Vertical, F.Cu at (129.5, 103.1)
- added REF**: PinHeader_1x01_P2.54mm_Vertical, Connector_PinHeader_2.54mm:PinHeader_1x01_P2.54mm_Vertical, F.Cu at (137.2, 108.2)
- added REF**: PinHeader_1x01_P2.54mm_Vertical, Connector_PinHeader_2.54mm:PinHeader_1x01_P2.54mm_Vertical, F.Cu at (137.2, 100.6)
- added REF**: SolderJumper-2_P1.3mm_Open_TrianglePad1.0x1.5mm, Jumper:SolderJumper-2_P1.3mm_Open_TrianglePad1.0x1.5mm, F.Cu at (125.7, 136.6)
- added REF**: PinHeader_1x01_P2.54mm_Vertical, Connector_PinHeader_2.54mm:PinHeader_1x01_P2.54mm_Vertical, F.Cu at (132.1, 108.2)
- added REF**: PinHeader_1x01_P2.54mm_Vertical, Connector_PinHeader_2.54mm:PinHeader_1x01_P2.54mm_Vertical, F.Cu at (139.7, 103.1)
- added REF**: PinHeader_1x01_P2.54mm_Vertical, Connector_PinHeader_2.54mm:PinHeader_1x01_P2.54mm_Vertical, F.Cu at (129.5, 110.7)
- added REF**: SolderJumper-2_P1.3mm_Open_TrianglePad1.0x1.5mm, Jumper:SolderJumper-2_P1.3mm_Open_TrianglePad1.0x1.5mm, F.Cu at (129.0, 120.4)
- added REF**: PinHeader_1x01_P2.54mm_Vertical, Connector_PinHeader_2.54mm:PinHeader_1x01_P2.54mm_Vertical, F.Cu at (129.5, 115.8)
- added REF**: SolderJumper-2_P1.3mm_Open_TrianglePad1.0x1.5mm, Jumper:SolderJumper-2_P1.3mm_Open_TrianglePad1.0x1.5mm, F.Cu at (125.7, 130.6)
- added REF**: PinHeader_1x01_P2.54mm_Vertical, Connector_PinHeader_2.54mm:PinHeader_1x01_P2.54mm_Vertical, F.Cu at (127.0, 100.6)
- added REF**: PinHeader_1x01_P2.54mm_Vertical, Connector_PinHeader_2.54mm:PinHeader_1x01_P2.54mm_Vertical, F.Cu at (144.8, 105.7)
- added REF**: PinHeader_1x01_P2.54mm_Vertical, Connector_PinHeader_2.54mm:PinHeader_1x01_P2.54mm_Vertical, F.Cu at (137.2, 110.7)
- added REF**: PinHeader_1x01_P2.54mm_Vertical, Connector_PinHeader_2.54mm:PinHeader_1x01_P2.54mm_Vertical, F.Cu at (134.6, 105.7)
- added REF**: PinHeader_1x01_P2.54mm_Vertical, Connector_PinHeader_2.54mm:PinHeader_1x01_P2.54mm_Vertical, F.Cu at (134.6, 103.1)
- added REF**: SolderJumper-2_P1.3mm_Open_TrianglePad1.0x1.5mm, Jumper:SolderJumper-2_P1.3mm_Open_TrianglePad1.0x1.5mm, F.Cu at (208.1, 119.0)
- added REF**: PinHeader_1x01_P2.54mm_Vertical, Connector_PinHeader_2.54mm:PinHeader_1x01_P2.54mm_Vertical, F.Cu at (127.0, 105.7)
- added REF**: PinHeader_1x01_P2.54mm_Vertical, Connector_PinHeader_2.54mm:PinHeader_1x01_P2.54mm_Vertical, F.Cu at (142.2, 100.6)
- added REF**: PinHeader_1x01_P2.54mm_Vertical, Connector_PinHeader_2.54mm:PinHeader_1x01_P2.54mm_Vertical, F.Cu at (139.7, 105.7)
- added REF**: PinHeader_1x01_P2.54mm_Vertical, Connector_PinHeader_2.54mm:PinHeader_1x01_P2.54mm_Vertical, F.Cu at (132.1, 98.0)
- added REF**: SolderJumper-2_P1.3mm_Open_TrianglePad1.0x1.5mm, Jumper:SolderJumper-2_P1.3mm_Open_TrianglePad1.0x1.5mm, F.Cu at (126.5, 66.7)
- added REF**: PinHeader_1x01_P2.54mm_Vertical, Connector_PinHeader_2.54mm:PinHeader_1x01_P2.54mm_Vertical, F.Cu at (134.6, 108.2)
- added REF**: PinHeader_1x01_P2.54mm_Vertical, Connector_PinHeader_2.54mm:PinHeader_1x01_P2.54mm_Vertical, F.Cu at (132.1, 110.7)
- added REF**: PinHeader_1x01_P2.54mm_Vertical, Connector_PinHeader_2.54mm:PinHeader_1x01_P2.54mm_Vertical, F.Cu at (124.5, 118.4)
- added REF**: PinHeader_1x01_P2.54mm_Vertical, Connector_PinHeader_2.54mm:PinHeader_1x01_P2.54mm_Vertical, F.Cu at (124.5, 108.2)
- added REF**: PinHeader_1x01_P2.54mm_Vertical, Connector_PinHeader_2.54mm:PinHeader_1x01_P2.54mm_Vertical, F.Cu at (127.0, 113.3)
- added REF**: PinHeader_1x01_P2.54mm_Vertical, Connector_PinHeader_2.54mm:PinHeader_1x01_P2.54mm_Vertical, F.Cu at (129.5, 100.6)
- added REF**: SolderJumper-2_P1.3mm_Open_TrianglePad1.0x1.5mm, Jumper:SolderJumper-2_P1.3mm_Open_TrianglePad1.0x1.5mm, F.Cu at (209.7, 82.9)
- added REF**: PinHeader_1x01_P2.54mm_Vertical, Connector_PinHeader_2.54mm:PinHeader_1x01_P2.54mm_Vertical, F.Cu at (142.2, 105.7)
- added REF**: PinHeader_1x01_P2.54mm_Vertical, Connector_PinHeader_2.54mm:PinHeader_1x01_P2.54mm_Vertical, F.Cu at (139.7, 110.7)
- added REF**: PinHeader_1x01_P2.54mm_Vertical, Connector_PinHeader_2.54mm:PinHeader_1x01_P2.54mm_Vertical, F.Cu at (124.5, 98.0)
- added REF**: SolderJumper-2_P1.3mm_Open_TrianglePad1.0x1.5mm, Jumper:SolderJumper-2_P1.3mm_Open_TrianglePad1.0x1.5mm, B.Cu at (169.5, 59.4)
- added REF**: SolderJumper-2_P1.3mm_Open_TrianglePad1.0x1.5mm, Jumper:SolderJumper-2_P1.3mm_Open_TrianglePad1.0x1.5mm, B.Cu at (159.3, 59.4)
- added REF**: PinHeader_1x01_P2.54mm_Vertical, Connector_PinHeader_2.54mm:PinHeader_1x01_P2.54mm_Vertical, F.Cu at (129.5, 98.0)
- added REF**: SolderJumper-2_P1.3mm_Open_TrianglePad1.0x1.5mm, Jumper:SolderJumper-2_P1.3mm_Open_TrianglePad1.0x1.5mm, B.Cu at (160.6, 154.7)
- added REF**: SolderJumper-2_P1.3mm_Open_TrianglePad1.0x1.5mm, Jumper:SolderJumper-2_P1.3mm_Open_TrianglePad1.0x1.5mm, B.Cu at (139.7, 154.7)
- added REF**: SolderJumper-2_P1.3mm_Open_TrianglePad1.0x1.5mm, Jumper:SolderJumper-2_P1.3mm_Open_TrianglePad1.0x1.5mm, B.Cu at (197.9, 154.7)
- added REF**: SolderJumper-2_P1.3mm_Open_TrianglePad1.0x1.5mm, Jumper:SolderJumper-2_P1.3mm_Open_TrianglePad1.0x1.5mm, B.Cu at (137.2, 59.4)
- added REF**: SolderJumper-2_P1.3mm_Open_TrianglePad1.0x1.5mm, Jumper:SolderJumper-2_P1.3mm_Open_TrianglePad1.0x1.5mm, B.Cu at (192.7, 59.4)
- added REF**: SolderJumper-2_P1.3mm_Open_TrianglePad1.0x1.5mm, Jumper:SolderJumper-2_P1.3mm_Open_TrianglePad1.0x1.5mm, B.Cu at (185.2, 59.4)
- added REF**: SolderJumper-2_P1.3mm_Open_TrianglePad1.0x1.5mm, Jumper:SolderJumper-2_P1.3mm_Open_TrianglePad1.0x1.5mm, B.Cu at (180.3, 154.7)
- added REF**: SolderJumper-2_P1.3mm_Open_TrianglePad1.0x1.5mm, Jumper:SolderJumper-2_P1.3mm_Open_TrianglePad1.0x1.5mm, B.Cu at (178.0, 59.4)
- added REF**: SolderJumper-2_P1.3mm_Open_TrianglePad1.0x1.5mm, Jumper:SolderJumper-2_P1.3mm_Open_TrianglePad1.0x1.5mm, B.Cu at (205.1, 67.4)
- added REF**: SolderJumper-2_P1.3mm_Open_TrianglePad1.0x1.5mm, Jumper:SolderJumper-2_P1.3mm_Open_TrianglePad1.0x1.5mm, B.Cu at (201.0, 59.4)
- added REF**: PinHeader_1x01_P2.54mm_Vertical, Connector_PinHeader_2.54mm:PinHeader_1x01_P2.54mm_Vertical, F.Cu at (129.5, 113.3)
- added REF**: PinHeader_1x01_P2.54mm_Vertical, Connector_PinHeader_2.54mm:PinHeader_1x01_P2.54mm_Vertical, F.Cu at (139.7, 100.6)
- TP35, TP37: footprint TestPoint:TestPoint_Pad_1.5x1.5mm -> TestPoint:TestPoint_THTPad_2.0x2.0mm_Drill1.0mm
- moved TP68 94.6 mm to (205.7, 126.4)
- moved TP94 8.03 mm to (172.7, 126.4)
- moved J3 3.83 mm to (167.6, 80.5)
- moved TP61 3.19 mm to (125.7, 70.5)
- moved J4 3.18 mm to (167.6, 72.9)
- moved J6 3.18 mm to (168.9, 140.3)
- moved TP101 3.18 mm to (162.6, 150.5)
- moved TP103 3.18 mm to (160.0, 146.7)
- moved TP105 3.18 mm to (157.5, 150.5)
- moved TP107 3.18 mm to (154.9, 146.7)
- moved TP109 3.18 mm to (152.4, 150.5)
- moved TP111 3.18 mm to (149.9, 146.7)
- moved TP113 3.18 mm to (147.3, 150.5)
- moved TP115 3.18 mm to (144.8, 146.7)
- moved TP117 3.18 mm to (142.2, 150.5)
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Routing:
- net GND: track 979.3 -> 1267.3 mm, vias 5 -> 7
- net /VDD_1V8: track 48.5 -> 83.1 mm
- net +2V5: track 43.9 -> 70.8 mm
- net Net-(J1-Pad63): track 48.2 -> 58.0 mm
- net Net-(J1-Pad61): track 47.0 -> 56.0 mm
- net Net-(J1-Pad62): track 47.1 -> 54.7 mm
- net Net-(J1-Pad64): track 48.1 -> 52.7 mm
- net /VCCIO0/1: track 22.3 -> 26.6 mm
- net /IOB91A: track 59.1 -> 62.0 mm
- net /IOB91B: track 54.5 -> 57.0 mm
- net /IOL14B: track 45.7 -> 43.9 mm
- net +5V: track 61.6 -> 63.2 mm, vias 1 -> 0
- net +3V3: track 47.7 -> 46.1 mm, vias 1 -> 0
- net /IOL3B: track 41.2 -> 39.8 mm
- net /IOL14A: track 48.9 -> 47.5 mm
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Other:
- outline, holes or cut-outs redrawn
- board text added: "DONE"
- board text added: "GND"
- board text added: "IOB12B"
- board text added: "IOB14B"
- board text added: "IOB24A"
- board text added: "IOB26A"
- board text added: "IOB26B"
- board text added: "IOB4A"
- board text added: "IOB4B"
- board text added: "IOB56A"
- board text added: "IOB56B"
- board text added: "IOB60A"
- board text added: "IOB89A"
- board text added: "IOB89B"
- board text added: "IOB91A"
- board text added: "IOB91B"
- board text added: "IOL12A"
- board text added: "IOL12B"
- board text added: "IOL14A"
- board text added: "IOL14B"
- board text added: "IOL3A"
- board text added: "IOL3B"
- board text added: "IOL5A"
- board text added: "IOL5B"
- board text added: "IOL9A"
- board text added: "IOL9B"
- board text added: "IOR18A"
- board text added: "IOR18B"
- board text added: "IOR20A"
- board text added: "IOR20B"
- board text added: "IOR22A"
- board text added: "IOR22B"
- board text added: "IOR24A"
- board text added: "IOR24B"
- board text added: "IOR31A"
- board text added: "IOR31B"
- board text added: "IOR33A"
- board text added: "IOR33B"
- board text added: "IOT11A"
- board text added: "IOT11B"
- board text added: "IOT15A"
- board text added: "IOT15B"
- board text added: "IOT19A"
- board text added: "IOT19B"
- board text added: "IOT1A"
- board text added: "IOT1B"
- board text added: "IOT21A"
- board text added: "IOT21B"
- board text added: "IOT23A"
- board text added: "IOT23B"
- board text added: "IOT31A"
- board text added: "IOT31B"
- board text added: "IOT3A"
- board text added: "IOT56A"
- board text added: "IOT56B"
- board text added: "IOT58A"
- board text added: "IOT58B"
- board text added: "IOT61A"
- board text added: "IOT61B"
- board text added: "IOT63A"
- board text added: "IOT63B"
- board text added: "IOT66A"
- board text added: "IOT66B"
- board text added: "IOT68A"
- board text added: "IOT68B"
- board text added: "IOT72A"
- board text added: "IOT72B"
- board text added: "IOT7A"
- board text added: "IOT7B"
- board text added: "M0_CKN"
- board text added: "M0_CKP"
- board text added: "M0_D0N"
- board text added: "M0_D0P"
- board text added: "M0_D1N"
- board text added: "M0_D1P"
- board text added: "M0_D2N"
- board text added: "M0_D2P"
- board text added: "M0_D3N"
- board text added: "M0_D3P"
- board text added: "READY"
- board text added: "RECONFIG"
- board text added: "TCK"
- board text added: "TDI"
- board text added: "TDO"
- board text added: "TMS"
- board text added: "VCCIO 0/1"
- board text added: "VCCIO 2/3"
- board text added: "VCCIO 6/7"
