File: ds_test_board_v3/ds_test_board3/ds_test_board3.kicad_pcb (KiCad board)
At the start: 2 copper layers, 91.4 x 100 mm, 203 parts, among them J1 DF40C-60DP-0.4V_51_, J2 DF40C-60DP-0.4V_51_, J3 Conn_01x30, J4 Conn_01x30, J5 Conn_01x30, J6 Conn_01x30

Commit message: 0315
Parts:
- added TP93: TestPoint, TestPoint:TestPoint_Pad_1.5x1.5mm, F.Cu at (170.6, 146.7)
- added TP94: TestPoint, TestPoint:TestPoint_Pad_1.5x1.5mm, F.Cu at (175.3, 121.9)
- TP101, TP103, TP105, TP107, TP109, TP111, TP113, TP115, TP117, TP119, TP121, TP123, TP125, TP128, TP66, TP67, TP69, TP71, TP73, TP75, TP77, TP79, TP81, TP83, TP85, TP87, TP89, TP91, TP93, TP95, TP99: footprint TestPoint:TestPoint_THTPad_1.5x1.5mm_Drill0.7mm -> TestPoint:TestPoint_Pad_1.5x1.5mm
- TP35, TP37: footprint TestPoint:TestPoint_THTPad_2.0x2.0mm_Drill1.0mm -> TestPoint:TestPoint_Pad_1.5x1.5mm
- moved TP92 5.12 mm to (177.8, 126.4)
- moved TP68 4.44 mm to (205.7, 121.9)
- moved TP70 4.44 mm to (203.2, 126.4)
- moved TP72 4.44 mm to (200.7, 121.9)
- moved TP74 4.44 mm to (198.1, 126.4)
- moved TP76 4.44 mm to (195.6, 121.9)
- moved TP78 4.44 mm to (193.0, 126.4)
- moved TP80 4.44 mm to (190.5, 121.9)
- moved TP82 4.44 mm to (188.0, 126.4)
- moved TP84 4.44 mm to (185.4, 121.9)
- moved TP86 4.44 mm to (182.9, 126.4)
- moved TP88 4.44 mm to (180.3, 121.9)
- turned J1 to 0 degrees
Connections:
- J1 pad 3: /IOT31A -> /IOR31A
- J1 pad 5: /IOT31B -> /IOR31B
- J1 pad 7: /IOT56A -> /IOB56A
- J1 pad 9: /IOT56B -> /IOB56B
- J5 pad 10: /IOT15A -> /IOB56A
- J5 pad 11: /IOT19B -> /IOB56B
- J5 pad 12: /IOT19A -> /IOB60A
- J5 pad 13: /IOT21B -> /DONE
- J5 pad 14: /IOT21A -> GND
- J5 pad 15: /IOT23B -> /VCCIO6/7
- J5 pad 16: /IOT23A -> /VCCIO6/7
- J5 pad 17: GND -> /IOT1A
- J5 pad 18: /VCCIO0/1 -> /IOT1B
- J5 pad 19: /VCCIO0/1 -> /IOT3A
- J5 pad 2: /IOL14B -> /IOR31A
- J5 pad 20: /IOT72B -> /IOT3B
- J5 pad 21: /IOT72A -> /IOT7A
- J5 pad 22: /IOT68B -> /IOT7B
- J5 pad 23: /IOT68A -> GND
- J5 pad 24: /IOT66B -> /IOL9A
- J5 pad 25: /IOT66A -> /IOL9B
- J5 pad 26: /IOT63B -> /IOL5A
- J5 pad 27: /IOT63A -> /IOL5B
- J5 pad 28: /IOT61B -> /IOL12A
- J5 pad 29: /IOT61A -> /IOL12B
- J5 pad 3: /IOL14A -> /IOR31B
- J5 pad 4: /IOL3B -> /IOB56A
- J5 pad 5: /IOL3A -> /IOB56B
- J5 pad 6: GND -> /IOT58A
- J5 pad 7: /IOT11B -> /IOT58B
- J5 pad 8: /IOT11A -> GND
- J5 pad 9: /IOT15B -> /READY
- J6 pad 10: /IOT7A -> /IOT72A
- J6 pad 11: /IOT3B -> /IOT72B
- J6 pad 12: /IOT3A -> /VCCIO0/1
- J6 pad 13: /IOT1B -> /VCCIO0/1
- J6 pad 14: /IOT1A -> GND
- J6 pad 15: /VCCIO6/7 -> /IOT23A
- J6 pad 16: /VCCIO6/7 -> /IOT23B
- J6 pad 17: GND -> /IOT21A
- J6 pad 18: /DONE -> /IOT21B
- J6 pad 19: /IOB60A -> /IOT19A
- J6 pad 2: /IOL12B -> /IOT61A
- J6 pad 20: /IOB56B -> /IOT19B
- J6 pad 21: /IOB56A -> /IOT15A
- J6 pad 22: /READY -> /IOT15B
- J6 pad 23: GND -> /IOT11A
- J6 pad 24: /IOT58B -> /IOT11B
- J6 pad 25: /IOT58A -> GND
- J6 pad 26: /IOT56B -> /IOL3A
- J6 pad 27: /IOT56A -> /IOL3B
- J6 pad 28: /IOT31B -> /IOL14A
- J6 pad 29: /IOT31A -> /IOL14B
- J6 pad 3: /IOL12A -> /IOT61B
- J6 pad 4: /IOL5B -> /IOT63A
- J6 pad 5: /IOL5A -> /IOT63B
- J6 pad 6: /IOL9B -> /IOT66A
- J6 pad 7: /IOL9A -> /IOT66B
- J6 pad 8: GND -> /IOT68A
- J6 pad 9: /IOT7B -> /IOT68B
- REF** pad 1: Net-(J1-Pad62) -> Net-(J1-Pad64)
- REF** pad 2: Net-(J1-Pad61) -> Net-(J1-Pad63) (x2)
- REF** pad 2: GND -> /IOT58A (x2)
- REF** pad 1: Net-(J1-Pad64) -> Net-(J1-Pad62) (x2)
- TP100 pad 1: /IOT21A -> GND
- TP101 pad 1: /IOT1B -> /VCCIO0/1
- TP102 pad 1: /IOT21B -> /DONE
- TP103 pad 1: /IOT3A -> /VCCIO0/1
- TP104 pad 1: /IOT19A -> /IOB60A
- TP105 pad 1: /IOT3B -> /IOT72B
- TP106 pad 1: /IOT19B -> /IOB56B
- TP107 pad 1: /IOT7A -> /IOT72A
- TP108 pad 1: /IOT15A -> /IOB56A
- TP109 pad 1: /IOT7B -> /IOT68B
- TP110 pad 1: /IOT15B -> /READY
- TP111 pad 1: GND -> /IOT68A
- TP112 pad 1: /IOT11A -> GND
- TP113 pad 1: /IOL9A -> /IOT66B
- TP114 pad 1: /IOT11B -> /IOT58B
- TP115 pad 1: /IOL9B -> /IOT66A
- TP116 pad 1: GND -> /IOT58A
- TP117 pad 1: /IOL5A -> /IOT63B
- TP118 pad 1: /IOL3A -> /IOB56B
- TP119 pad 1: /IOL5B -> /IOT63A
- TP120 pad 1: /IOL3B -> /IOB56A
- TP121 pad 1: /IOL12A -> /IOT61B
- TP122 pad 1: /IOL14A -> /IOR31B
- TP123 pad 1: /IOL12B -> /IOT61A
- TP124 pad 1: /IOL14B -> /IOR31A
- TP127 pad 1: Net-(J1-Pad64) -> Net-(J1-Pad62)
- TP128 pad 1: Net-(J1-Pad63) -> Net-(J1-Pad61)
- TP65 pad 1: Net-(J1-Pad61) -> Net-(J1-Pad63)
- TP66 pad 1: Net-(J1-Pad62) -> Net-(J1-Pad64)
- TP69 pad 1: /IOT31A -> /IOL14B
- TP70 pad 1: /IOT61A -> /IOL12B
- TP71 pad 1: /IOT31B -> /IOL14A
- TP72 pad 1: /IOT61B -> /IOL12A
- TP73 pad 1: /IOT56A -> /IOL3B
- TP74 pad 1: /IOT63A -> /IOL5B
- TP75 pad 1: /IOT56B -> /IOL3A
- TP76 pad 1: /IOT63B -> /IOL5A
- TP77 pad 1: /IOT58A -> GND
- TP78 pad 1: /IOT66A -> /IOL9B
- TP79 pad 1: /IOT58B -> /IOT11B
- TP80 pad 1: /IOT66B -> /IOL9A
- TP81 pad 1: GND -> /IOT11A
- TP82 pad 1: /IOT68A -> GND
- TP83 pad 1: /READY -> /IOT15B
- TP84 pad 1: /IOT68B -> /IOT7B
- TP85 pad 1: /IOB56A -> /IOT15A
- TP86 pad 1: /IOT72A -> /IOT7A
- TP87 pad 1: /IOB56B -> /IOT19B
- TP88 pad 1: /IOT72B -> /IOT3B
- TP89 pad 1: /IOB60A -> /IOT19A
- TP91 pad 1: /DONE -> /IOT21B
- TP92 pad 1: /VCCIO0/1 -> /IOT3A
- TP93 pad 1: GND -> /IOT21A
- TP94 pad 1: GND -> /IOT1A
- TP95 pad 1: /VCCIO6/7 -> /IOT23A
- TP96 pad 1: /IOT23A -> /VCCIO6/7
- TP98 pad 1: /IOT23B -> /VCCIO6/7
- TP99 pad 1: /IOT1A -> GND
Routing:
- net /VCCIO0/1: track 26.6 -> 90.1 mm, vias 1 -> 0
- net /IOT31A: track 56.8 -> 0.00 mm
- net /IOT56A: track 55.1 -> 0.00 mm
- net GND: track 1267.3 -> 1215.3 mm
- net /IOT31B: track 51.6 -> 0.00 mm
- net /IOT56B: track 49.8 -> 0.00 mm
- net /IOR31B: track 40.9 -> 88.4 mm, vias 1 -> 2
- net /IOR31A: track 38.8 -> 82.7 mm, vias 1 -> 2
- net /IOT1B: track 46.8 -> 9.14 mm
- net /IOT1A: track 41.6 -> 8.26 mm
- net /IOB56B: track 44.5 -> 72.7 mm, vias 0 -> 2
- net /IOT21A: track 20.9 -> 46.1 mm, vias 1 -> 0
- net /IOB56A: track 49.7 -> 73.6 mm, vias 0 -> 2
- net /IOT72B: track 29.1 -> 48.5 mm, vias 1 -> 0
- net /IOT3B: track 48.5 -> 29.1 mm, vias 0 -> 1
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
Commit message: 0315
Parts:
- removed the REF** at (160.6, 154.7)
- removed the REF** at (139.7, 154.7)
- removed the REF** at (180.3, 154.7)
- removed TP99: TestPoint, TestPoint:TestPoint_Pad_1.5x1.5mm
- added REF**: SolderJumper-2_P1.3mm_Open_TrianglePad1.0x1.5mm, Jumper:SolderJumper-2_P1.3mm_Open_TrianglePad1.0x1.5mm, F.Cu at (136.4, 154.7)
- added REF**: SolderJumper-2_P1.3mm_Open_TrianglePad1.0x1.5mm, Jumper:SolderJumper-2_P1.3mm_Open_TrianglePad1.0x1.5mm, F.Cu at (179.2, 154.6)
- added REF**: SolderJumper-2_P1.3mm_Open_TrianglePad1.0x1.5mm, Jumper:SolderJumper-2_P1.3mm_Open_TrianglePad1.0x1.5mm, F.Cu at (210.2, 113.0)
- added TP95: TestPoint, TestPoint:TestPoint_THTPad_1.5x1.5mm_Drill0.7mm, F.Cu at (165.1, 146.7)
- REF**: moved to F.Cu
- TP101, TP103, TP105, TP107, TP109, TP111, TP113, TP115, TP117, TP119, TP121, TP123, TP125, TP127, TP128, TP35, TP37, TP67, TP69, TP71, TP73, TP75, TP77, TP79, TP81, TP83, TP85, TP87, TP89, TP91, TP93 (x2), TP95: footprint TestPoint:TestPoint_Pad_1.5x1.5mm -> TestPoint:TestPoint_THTPad_1.5x1.5mm_Drill0.7mm
- turned REF** to 0 degrees
Connections:
- J1 pad 3: /IOR31A -> IOT31A
- J1 pad 5: /IOR31B -> IOT31B
- J1 pad 7: /IOB56A -> IOT56A
- J1 pad 9: /IOB56B -> IOT56B
- J5 pad 2: /IOR31A -> IOT31A
- J5 pad 3: /IOR31B -> IOT31B
- J5 pad 4: /IOB56A -> IOT56A
- J5 pad 5: /IOB56B -> IOT56B
- TP118 pad 1: /IOB56B -> IOT56B
- TP120 pad 1: /IOB56A -> IOT56A
- TP122 pad 1: /IOR31B -> IOT31B
- TP124 pad 1: /IOR31A -> IOT31A
Routing:
- net GND: track 1215.3 -> 1264.2 mm
- net /IOR31B: track 88.4 -> 40.9 mm, vias 2 -> 1
- net IOT31B: track 0.00 -> 47.4 mm, vias 0 -> 1
- net /IOB56B: track 72.7 -> 27.6 mm, vias 2 -> 1
- net IOT56B: track 0.00 -> 44.8 mm, vias 0 -> 1
- net IOT31A: track 0.00 -> 43.9 mm, vias 0 -> 1
- net /IOR31A: track 82.7 -> 38.8 mm, vias 2 -> 1
- net IOT56A: track 0.00 -> 39.8 mm, vias 0 -> 1
- net /IOB56A: track 73.6 -> 34.4 mm, vias 2 -> 1
- net /IOT1A: track 8.26 -> 30.3 mm, vias 0 -> 1
- net /IOT1B: track 9.14 -> 21.9 mm, vias 0 -> 1
- net /IOT3A: track 26.7 -> 36.6 mm
- net /IOT3B: track 29.1 -> 34.8 mm
- net /IOT7A: track 36.7 -> 40.2 mm
- net Net-(J1-Pad63): track 65.8 -> 68.8 mm
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
Commit message: 0315
Parts:
- TP66: footprint TestPoint:TestPoint_Pad_1.5x1.5mm -> TestPoint:TestPoint_THTPad_1.5x1.5mm_Drill0.7mm
Connections:
- REF** pad 1: Net-(J1-Pad63) -> Net-(J1-Pad61) (x2)
- REF** pad 2: /IOT58A -> GND (x2)
Routing:
- net /IOT58A: track 67.9 -> 39.1 mm, vias 3 -> 2
- net Net-(J1-Pad63): track 68.8 -> 59.0 mm
- net Net-(J1-Pad61): track 48.2 -> 58.0 mm
- net GND: track 1264.2 -> 1268.8 mm
Changed lines of the file:
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@@
 			(size 0.3 0.3)
 			(layers "F.Cu" "F.Mask")
-			(net 45 "Net-(J1-Pad63)")
+			(net 47 "Net-(J1-Pad61)")
 			(zone_connect 2)
 			(options
@@
 			(size 0.3 0.3)
 			(layers "F.Cu" "F.Mask")
-			(net 45 "Net-(J1-Pad63)")
+			(net 47 "Net-(J1-Pad61)")
 			(zone_connect 2)
 			(options
@@
 			(size 0.3 0.3)
 			(layers "F.Cu" "F.Mask")
-			(net 53 "/IOT58A")
+			(net 50 "GND")
 			(zone_connect 2)
 			(options
@@
 		)
 	)
-	(footprint "TestPoint:TestPoint_Pad_1.5x1.5mm"
+	(footprint "TestPoint:TestPoint_THTPad_1.5x1.5mm_Drill0.7mm"
 		(layer "F.Cu")
 		(at 210.185 142.875)
-		(descr "SMD rectangular pad as test Point, square 1.5mm side length")
-		(tags "test point SMD pad rectangle square")
+		(descr "THT rectangular pad as test Point, square 1.5mm side length, hole diameter 0.7mm")
+		(tags "test point THT pad rectangle square")
 		(property "Reference" "TP66"
 			(at 0 -1.648 0)
@@
 			)
 		)
-		(property ki_fp_filters "Pin* Test*")
-		(sheetname "ルート")
-		(sheetfile "ds_test_board3.kicad_sch")
-		(attr exclude_from_pos_files)
+		(attr exclude_from_pos_files exclude_from_bom)
 		(fp_line
 			(start -0.95 -0.95)
@@
 			)
 		)
-		(pad "1" smd rect
+		(pad "1" thru_hole rect
 			(at 0 0)
 			(size 1.5 1.5)
-			(layers "F.Cu" "F.Mask")
+			(drill 0.7)
+			(layers "*.Cu" "*.Mask")
+			(remove_unused_layers no)
 			(net 44 "Net-(J1-Pad64)")
 			(pinfunction "1")
@@
 			(size 0.3 0.3)
 			(layers "F.Cu" "F.Mask")
-			(net 53 "/IOT58A")
+			(net 50 "GND")
 			(zone_connect 2)
 			(options
@@
 	)
 	(segment
-		(start 125.73 137.34)
-		(end 125.73 142.24)
-		(width 0.25)
-		(layer "F.Cu")
-		(net 45)
-	)
-	(segment
 		(start 210.185 116.7384)
 		(end 210.185 116.6114)
@@
 	)
 	(segment
-		(start 125.73 144.272)
-		(end 125.73 142.24)
-		(width 0.25)
-		(layer "F.Cu")
-		(net 45)
-	)
-	(segment
 		(start 210.185 116.6114)
 		(end 210.2104 116.586)
@@
 		(start 210.2104 116.586)
 		(end 210.2104 113.7688)
-		(width 0.15)
-		(layer "F.Cu")
-		(net 45)
-	)
-	(segment
-		(start 127.762 146.304)
-		(end 125.73 144.272)
 		(width 0.25)
 		(layer "F.Cu")
@@
 	)
 	(segment
+		(start 125.73 137.34)
+		(end 125.73 142.24)
+		(width 0.25)
+		(layer "F.Cu")
+		(net 47)
+	)
+	(segment
+		(start 125.73 144.272)
+		(end 125.73 142.24)
+		(width 0.25)
+		(layer "F.Cu")
+		(net 47)
+	)
+	(segment
+		(start 127.762 146.304)
+		(end 125.73 144.272)
+		(width 0.25)
+		(layer "F.Cu")
+		(net 47)
+	)
+	(segment
 		(start 153.64 114.33)
 		(end 125.73 142.24)
@@
 		(start 132.08 146.304)
 		(end 132.08 141.994)
-		(width 0.15)
+		(width 0.25)
 		(layer "F.Cu")
 		(net 50)
@@
 		(start 133.1976 154.686)
 		(end 135.673 154.686)
-		(width 0.15)
+		(width 0.25)
 		(layer "F.Cu")
 		(net 50)
@@
 		(start 132.08 150.495)
 		(end 132.08 146.304)
-		(width 0.15)
+		(width 0.25)
 		(layer "F.Cu")
 		(net 50)
@@
 		(start 132.08 150.495)
 		(end 132.08 153.5684)
-		(width 0.15)
+		(width 0.25)
+		(layer "F.Cu")
+		(net 50)
+	)
+	(segment
+		(start 125.73 135.89)
+		(end 125.73 131.281)
+		(width 0.25)
 		(layer "F.Cu")
 		(net 50)
@@
 		(start 132.08 153.5684)
 		(end 133.1976 154.686)
-		(width 0.15)
+		(width 0.25)
 		(layer "F.Cu")
 		(net 50)
@@
 		(start 130.7592 66.2686)
 		(end 130.7592 74.5362)
-		(width 0.15)
+		(width 0.25)
 		(layer "F.Cu")
 		(net 50)
@@
 	)
 	(segment
-		(start 125.73 131.281)
-		(end 128.995 131.281)
-		(width 0.25)
-		(layer "F.Cu")
-		(net 53)
-	)
-	(segment
 		(start 155.956 107.95)
 		(end 156.464 107.95)
@@
 	)
 	(segment
-		(start 125.73 135.89)
-		(end 125.73 131.281)
-		(width 0.25)
-		(layer "F.Cu")
-		(net 53)
-	)
-	(segment
-		(start 128.995 131.281)
-		(end 129.032 131.318)
-		(width 0.25)
-		(layer "F.Cu")
-		(net 53)
-	)
-	(segment
 		(start 144.78 131.31)
 		(end 144.78 121.92)
@@
 	)
 	(via
-		(at 129.032 131.318)
-		(size 0.5)
-		(drill 0.3)
-		(layers "F.Cu" "B.Cu")
-		(net 53)
-	)
-	(via
 		(at 144.78 119.126)
 		(size 0.5)
@@
 	)
 	(segment
-		(start 132.588 131.318)
-		(end 129.032 131.318)
-		(width 0.15)
-		(layer "B.Cu")
-		(net 53)
-	)
-	(segment
 		(start 163.7538 109.2454)
 		(end 164.808 110.2996)
 		(width 0.15)
 		(layer "B.Cu")
-		(net 53)
-	)
-	(segment
-		(start 144.78 119.126)
-		(end 132.588 131.318)
-		(width 0.15)
-		(layer "B.Cu")
